File: CIB_Main_PCB/misc relays.kicad_sch (KiCad schematic)
At the start: 7 parts, among them U3 ULN2803A, U4 MCP23017_SO, U6 ULN2803A, U7 MCP23017_SO, U8 ULN2803A

Commit message: added snubbing to the relays
Connections:
- net DUT Power Relay 1: now also U3.11 (O8); no longer U3.18 (O1)
- net DUT Power Relay 2: now also U3.12 (O7); no longer U3.17 (O2)
- net External Relay 1: now also U3.18 (O1); no longer U3.16 (O3)
- net External Relay 2: now also U3.17 (O2); no longer U3.15 (O4)
- net External Relay 3: now also U3.16 (O3); no longer U3.14 (O5)
- net External Relay 4: now also U3.15 (O4); no longer U3.13 (O6)
- net External Relay 5: now also U3.14 (O5); no longer U3.12 (O7)
- net External Relay 6: now also U3.13 (O6); no longer U3.11 (O8)
- net PT100 PT1000 Simulation/Relay 1: now also U6.12 (O7); no longer U6.14 (O5)
- net PT100 PT1000 Simulation/Relay 2: now also U6.13 (O6); no longer U6.15 (O4)
- net PT100 PT1000 Simulation/Relay 3: now also U6.14 (O5); no longer U6.16 (O3)
- net PT100 PT1000 Simulation/Relay 4: now also U6.15 (O4); no longer U6.17 (O2)
- net PT100 PT1000 Simulation/Relay 5: now also U6.16 (O3); no longer U6.18 (O1)
- net RAG Relays/Relay 1: now also U6.18 (O1); no longer U6.12 (O7)
- net RAG Relays/Relay 2: now also U6.17 (O2); no longer U6.13 (O6)
- net at U8.1 (I1): now also U4.28 (GPA7); no longer U4.21 (GPA0)
- net at U8.2 (I2): now also U4.27 (GPA6); no longer U4.22 (GPA1)
- net at U8.3 (I3): now also U4.26 (GPA5); no longer U4.23 (GPA2)
- net at U8.4 (I4): now also U4.25 (GPA4); no longer U4.24 (GPA3)
- net at U8.5 (I5): now also U4.24 (GPA3); no longer U4.25 (GPA4)
- net at U8.6 (I6): now also U4.23 (GPA2); no longer U4.26 (GPA5)
- net at U8.7 (I7): now also U4.22 (GPA1); no longer U4.27 (GPA6)
- net at U8.8 (I8): now also U4.21 (GPA0); no longer U4.28 (GPA7)
