File: CIB_Main_PCB - Mimic Octopus/MicroControler Interface.kicad_sch (KiCad schematic)
At the start: 13 parts, among them J17 LabJack1, J18 Labjack2

Commit message: BoM
Parts:
- J17, J18: Height (none) -> 16; Manufacturer_Part_Number 1848765 -> (none); Mouser # (none) -> 651-1848765; Mouser Part Number 651-1848765 -> (none)
- XA1: dnp (none) -> dnp
Changed lines of the file:
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@@
       (effects (font (size 1.524 1.524)) hide)
+    )
+    (property "dnp" "dnp" (id 4) (at 119.38 80.01 0)
+      (effects (font (size 1.27 1.27)) hide)
     )
     (pin "3V3")
@@
       (effects (font (size 1.27 1.27)) hide)
     )
-    (property "Mouser Part Number" "651-1848765" (id 8) (at 48.26 71.12 0)
+    (property "Mouser Part Number" "" (id 8) (at 48.26 71.12 0)
       (effects (font (size 1.27 1.27)) (justify left) hide)
     )
@@
       (effects (font (size 1.27 1.27)) (justify left) hide)
     )
-    (property "Manufacturer_Part_Number" "1848765" (id 14) (at 48.26 68.58 0)
-      (effects (font (size 1.27 1.27)) (justify left) hide)
+    (property "Manufacturer_Part_Number" "" (id 14) (at 48.26 68.58 0)
+      (effects (font (size 1.27 1.27)) (justify left) hide)
+    )
+    (property "Height" "16" (id 15) (at 29.21 58.42 0)
+      (effects (font (size 1.27 1.27)) hide)
+    )
+    (property "Mouser #" "651-1848765" (id 16) (at 29.21 58.42 0)
+      (effects (font (size 1.27 1.27)) hide)
     )
     (pin "1")
@@
       (effects (font (size 1.27 1.27)) hide)
     )
-    (property "Mouser Part Number" "651-1848765" (id 8) (at 48.26 124.46 0)
+    (property "Mouser Part Number" "" (id 8) (at 48.26 124.46 0)
       (effects (font (size 1.27 1.27)) (justify left) hide)
     )
@@
       (effects (font (size 1.27 1.27)) (justify left) hide)
     )
-    (property "Manufacturer_Part_Number" "1848765" (id 14) (at 48.26 121.92 0)
-      (effects (font (size 1.27 1.27)) (justify left) hide)
-    )
-    (pin "1")
+    (property "Manufacturer_Part_Number" "" (id 14) (at 48.26 121.92 0)
+      (effects (font (size 1.27 1.27)) (justify left) hide)
+    )
+    (property "Height" "16" (id 15) (at 29.21 111.76 0)
+      (effects (font (size 1.27 1.27)) hide)
+    )
+    (property "Mouser #" "651-1848765" (id 16) (at 29.21 111.76 0)
+      (effects (font (size 1.27 1.27)) hide)
+    )
+    (pin "1")
