File: CIB_Main_PCB - Mimic Octopus/CIB PSU.kicad_sch (KiCad schematic)
At the start: 25 parts, among them U25 LM2672M-12, U9 5V Reg

Commit message: added changes
Parts:
- removed C12: 10nF, Capacitor_SMD:C_1206_3216Metric_Pad1.33x1.80mm_HandSolder, symbol Device:C_Small
- removed C14: 47uF 20 V, Capacitor_SMD:C_Elec_8x10.2, symbol Device:C_Polarized_Small
- removed D23: 50V, Diode_SMD:D_SMA_Handsoldering, symbol Device:D_Schottky
- removed L1: 52 Ω, ~, symbol Device:L_Coupled_Small
- removed L2: 68uH, Inductor_SMD:L_Pulse_PA4344, symbol Device:L_Small
- removed R1, R28, R4: 0, Resistor_SMD:R_2010_5025Metric_Pad1.40x2.65mm_HandSolder, symbol Device:R_Small
- removed U25: LM2672M-12, Package_SO:SOIC-8_3.9x4.9mm_P1.27mm, symbol Regulator_Switching:LM2672M-12
- added C21, C23, C30: 10uF 16 V, Capacitor_SMD:C_1206_3216Metric_Pad1.33x1.80mm_HandSolder, symbol Device:C_Small
- added C22, C24, C31: 22uF 16 V, Capacitor_SMD:C_1206_3216Metric_Pad1.33x1.80mm_HandSolder, symbol Device:C_Small
- added C25, C26, C27: 470uF 16 V, Capacitor_SMD:C_Elec_8x10.2, symbol Device:C_Polarized_Small
- added D20, D21, D22: Green, Diode_SMD:D_1206_3216Metric_Pad1.42x1.75mm_HandSolder, symbol Device:LED_Small_Filled
- added R45, R49: 5k1, Resistor_SMD:R_1206_3216Metric_Pad1.30x1.75mm_HandSolder, symbol Device:R_Small
- added R46: 1k2, Resistor_SMD:R_1206_3216Metric_Pad1.30x1.75mm_HandSolder, symbol Device:R_Small
- added R47: 330, Resistor_SMD:R_1206_3216Metric_Pad1.30x1.75mm_HandSolder, symbol Device:R_Small
- added R48: 120, Resistor_SMD:R_1206_3216Metric_Pad1.30x1.75mm_HandSolder, symbol Device:R_Small
- added U9: TSR 1-2433E, Connector_PinHeader_2.54mm:PinHeader_1x03_P2.54mm_Vertical, symbol Regulator_Linear:KA78M05_TO252
- U8: renamed from U9; value 5V Reg -> TSR 1-2450E; footprint Package_TO_SOT_SMD:TO-252-2 -> Connector_PinHeader_2.54mm:PinHeader_1x03_P2.54mm_Vertical; DigiKey # BA50BC0FP-E2CT-ND -> 1951-TSR1-2450E-ND; Manufacturer Rohm Semiconductor -> Traco Power; Manufacturer # BA50BC0FP-E2 -> TSR 1-2450E
- renumbered C21 to C11, C22 to C12, C23 to C13, C24 to C14, C25 to C15, C26 to C16, C27 to C17, C3 to C18, C11 to C19, C13 to C20, C1 to C28, C2 to C29, R50 to R43, R51 to R44
Connections:
- net +VDC is gone; now on net +12V: C18.1
- net Filtered supply is gone; now on net +12V: C19.1, C20.1
- net GND is gone; now on net -VDC: C11.2, C12.2, C13.2, C14.2, C15.2, C16.2, C17.2, C19.2, C20.2, C28.2, C29.2, D19.3 (A), R44.2, U8.2 (GND)
- net +12V: now also C21.1, C22.1, C27.1, R46.1, U9.1 (VI)
- net +5V: now also R45.1, R47.1
- net -VDC: now also C21.2, C22.2, C23.2, C24.2, C25.2, C26.2, C27.2, C30.2, C31.2, D20.1 (K), D21.1 (K), D22.1 (K), R49.2, U9.2 (GND)
- new net: D21.2 (A), R47.2
- new net: D22.2 (A), R48.2
- new net: D20.2 (A), R46.2
- new net +3V3: C23.1, C24.1, C25.1, C26.1, R48.1, U9.3 (VO)
- new net CIB 5V monitor: C30.1, C31.1, R45.2, R49.1
Other:
- note added: "Vout = Rbottom * Vin ---------- Rtop + Rbottom Vout = 0-2.5 VDC 5 VDC = 0-5 VDC"
- moved on the sheet: C11, C12, C13, C14, C15, C16, C17, C18, C19, C20, C28, C29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

Commit message: changes
Connections:
- net -VDC renamed GND
Changed lines of the file:
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@@
   (junction (at 68.58 45.72) (diameter 0) (color 0 0 0 0)
   )
-  (junction (at 52.07 63.5) (diameter 0) (color 0 0 0 0)
-  )
   (junction (at 170.18 82.55) (diameter 0) (color 0 0 0 0)
   )
@@
   (junction (at 46.99 138.43) (diameter 0) (color 0 0 0 0)
   )
-  (junction (at 36.83 63.5) (diameter 0) (color 0 0 0 0)
-  )
   (junction (at 154.94 45.72) (diameter 0) (color 0 0 0 0)
   )
@@
   )
   (wire (pts (xy 140.97 54.61) (xy 140.97 58.42))
-    (stroke (width 0) (type default) (color 0 0 0 0))
-  )
-  (wire (pts (xy 36.83 63.5) (xy 52.07 63.5))
     (stroke (width 0) (type default) (color 0 0 0 0))
   )
@@
     )
     (property "Datasheet" "" (id 3) (at 46.99 149.86 0)
-      (effects (font (size 1.27 1.27)) hide)
-    )
-    (pin "1")
-  )
-  (symbol (lib_id "power:-VDC") (at 36.83 63.5 180) (unit 1)
-    (in_bom yes) (on_board yes) (fields_autoplaced)
-    (property "Reference" "#PWR0104" (id 0) (at 36.83 60.96 0)
-      (effects (font (size 1.27 1.27)) hide)
-    )
-    (property "Value" "-VDC" (id 1) (at 36.83 71.12 0))
-    (property "Footprint" "" (id 2) (at 36.83 63.5 0)
-      (effects (font (size 1.27 1.27)) hide)
-    )
-    (property "Datasheet" "" (id 3) (at 36.83 63.5 0)
       (effects (font (size 1.27 1.27)) hide)
     )
@@
       (effects (font (size 1.27 1.27)) hide)
     )
+    (pin "1")
+  )
+  (symbol (lib_id "power:GND") (at 36.83 63.5 0) (unit 1)
+    (in_bom yes) (on_board yes) (fields_autoplaced)
+    (property "Reference" "#PWR0379" (id 0) (at 36.83 69.85 0)
+      (effects (font (size 1.27 1.27)) hide)
+    )
+    (property "Value" "GND" (id 1) (at 36.83 68.58 0))
+    (property "Footprint" "" (id 2) (at 36.83 63.5 0)
+      (effects (font (size 1.27 1.27)) hide)
+    )
+    (property "Datasheet" "" (id 3) (at 36.83 63.5 0)
+      (effects (font (size 1.27 1.27)) hide)
+    )

Commit message: V0.1 PCB to be sent out
Parts:
- removed U8: TSR 1-2450E, Connector_PinHeader_2.54mm:PinHeader_1x03_P2.54mm_Vertical, symbol Regulator_Linear:KA78M05_TO252
- removed U9: TSR 1-2433E, Connector_PinHeader_2.54mm:PinHeader_1x03_P2.54mm_Vertical, symbol Regulator_Linear:KA78M05_TO252
- added J3: CIB Power, Component Search Engine:Pluggable Terminal Blocks SDC 2.5mm pitch 4 Pin, symbol Component Search Engine:Pluggable Terminal Blocks SDC 2,5/ 4-PV-5,0 0-ZB
- added NT15: NetTie_2, NetTie:NetTie-2_SMD_Pad0.5mm, symbol Device:NetTie_2
- added PS1: TSR1-2450E, Component Search Engine:TSR12450E, symbol Component temp:TSR1-2450E
- added PS2: TSR1-2433E, Component Search Engine:TSR12433E, symbol Component temp:TSR1-2433E
- added R176, R177: 1k2, Resistor_SMD:R_1206_3216Metric_Pad1.30x1.75mm_HandSolder, symbol Device:R_Small
- added TP1: TP 5V0, TestPoint:TestPoint_Pad_D2.0mm, symbol Connector:TestPoint
- added TP2: TP 3V3, TestPoint:TestPoint_Pad_D2.0mm, symbol Connector:TestPoint
- added TP3: TP 12V3, TestPoint:TestPoint_Pad_D2.0mm, symbol Connector:TestPoint
- added TP4: TP GND, TestPoint:TestPoint_Pad_D2.0mm, symbol Connector:TestPoint
Connections:
- net +12V: now also J3.1, J3.3, NT15.2, PS1.1 (+VIN), PS2.1 (+VIN), TP3.1; no longer R43.1
- net +3V3: now also PS2.3 (+VOUT), TP2.1
- net +5V: now also PS1.3 (+VOUT), TP1.1
- net CIB 12V monitor: now also R176.2; no longer C28.1, C29.1, D19.1 (K), D19.2 (K), R43.2, R44.1
- net CIB 5V monitor: now also R177.2; no longer C30.1, C31.1, R45.2, R49.1
- net GND: now also J3.2, J3.4, PS1.2 (GND), PS2.2 (GND), TP4.1
- new net: C28.1, C29.1, D19.1 (K), D19.2 (K), R176.1, R43.2, R44.1
- new net: C30.1, C31.1, R177.1, R45.2, R49.1
- new net: NT15.1, R43.1
Other:
- moved on the sheet: C21, C22, C23, C24, C25, C26, C27

Commit message: BoM
Parts:
- C11, C13, C18, C19, C21, C23, C28, C30, D19: Height (none) -> 2
- C12, C14, C22, C24, C29, C31: DigiKey # 732-7642-1-ND -> 1276-3048-1-ND; DigiKey Price/Stock https://www.digikey.co.uk/en/products/detail/w%C3%BCrth-ele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 -> https://www.digikey.co.uk/en/products/detail/samsung-electr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; Height (none) -> 2; Manufacturer Würth Elektronik -> Samsung Electro-Mechanics; Manufacturer # 885012108018 -> CL31A226KOHNNNE
- C15, C16, C17, C25, C26, C27: value 470uF 16 V -> 470uF 20 V; DigiKey # 732-8526-1-ND -> P124165CT-ND; DigiKey Price/Stock https://www.digikey.co.uk/en/products/detail/w%C3%BCrth-ele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 -> https://www.digikey.co.uk/en/products/detail/panasonic-elec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; Height (none) -> 12; Manufacturer Würth Elektronik -> Panasonic Electronic; Manufacturer # 865060353009 -> (none)
- C20: value 100uF 30 V -> 100uF 25 V; DigiKey # 732-8526-1-ND -> P123675CT-ND; DigiKey Price/Stock https://www.digikey.co.uk/en/products/detail/w%C3%BCrth-ele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 -> https://www.digikey.co.uk/en/products/detail/panasonic-elec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; Height (none) -> 7; Manufacturer Würth Elektronik -> Panasonic Electronic; Manufacturer # 865060353009 -> (none)
- D20, D21, D22: DigiKey Price/Stock (none) -> https://www.digikey.co.uk/en/products/detail/w%C3%BCrth-ele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; Height (none) -> 2
- J3: Height (none) -> 16; Manufacturer_Part_Number 1864053 -> (none); Mouser # (none) -> 651-1864053; Mouser Part Number 651-1864053 -> (none)
- NT15, TP1, TP2, TP3, TP4: dnp (none) -> dnp
- PS1: DigiKey # (none) -> 1951-TSR1-2450E-ND; DigiKey Price/Stock (none) -> https://www.digikey.co.uk/en/products/detail/traco-power/TS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; Digikey Part Number 1951-TSR1-2450E-ND -> (none); Height 10.7 -> 11; Manufacturer (none) -> Traco Power; Manufacturer # (none) -> TSR1-2450E; Manufacturer_Name Traco Power -> (none); Manufacturer_Part_Number TSR1-2450E -> (none); Mouser # (none) -> TSR12450E
- PS2: DigiKey # (none) -> 1951-TSR1-2433E-ND; DigiKey Price/Stock (none) -> https://www.digikey.co.uk/en/products/detail/traco-power/TS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; Digikey Part Number 1951-TSR1-2433E-ND -> (none); Height 10.7 -> 11; Manufacturer (none) -> Traco Power; Manufacturer # (none) -> TSR1-2433E; Manufacturer_Name Traco Power -> (none); Manufacturer_Part_Number TSR1-2433E -> (none); Mouser # (none) -> TSR12433E

Commit message: changes
Parts:
- NT15: value NetTie_2 -> NetTie
Changed lines of the file:
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@@
   (symbol (lib_id "Device:C_Polarized_Small") (at 246.38 50.8 0) (unit 1)
     (in_bom yes) (on_board yes) (fields_autoplaced)
-    (property "Reference" "C16" (id 0) (at 249.682 48.9838 0)
-      (effects (font (size 1.27 1.27)) (justify left))
-    )
-    (property "Value" "470uF 20 V" (id 1) (at 249.682 51.5238 0)
+    (property "Reference" "C16" (id 0) (at 248.92 48.9838 0)
+      (effects (font (size 1.27 1.27)) (justify left))
+    )
+    (property "Value" "470uF 20 V" (id 1) (at 248.92 51.5238 0)
       (effects (font (size 1.27 1.27)) (justify left))
     )
@@
   (symbol (lib_id "Device:C_Polarized_Small") (at 140.97 101.6 0) (unit 1)
     (in_bom yes) (on_board yes) (fields_autoplaced)
-    (property "Reference" "C27" (id 0) (at 138.684 99.7838 0)
+    (property "Reference" "C27" (id 0) (at 138.43 99.7838 0)
       (effects (font (size 1.27 1.27)) (justify right))
     )
-    (property "Value" "470uF 20 V" (id 1) (at 138.684 102.3238 0)
+    (property "Value" "470uF 20 V" (id 1) (at 138.43 102.3238 0)
       (effects (font (size 1.27 1.27)) (justify right))
     )
@@
   (symbol (lib_id "Device:C_Small") (at 154.94 100.33 0) (unit 1)
     (in_bom yes) (on_board yes) (fields_autoplaced)
-    (property "Reference" "C21" (id 0) (at 158.496 99.0662 0)
-      (effects (font (size 1.27 1.27)) (justify left))
-    )
-    (property "Value" "10uF 16 V" (id 1) (at 158.496 101.6062 0)
+    (property "Reference" "C21" (id 0) (at 157.48 99.0662 0)
+      (effects (font (size 1.27 1.27)) (justify left))
+    )
+    (property "Value" "10uF 16 V" (id 1) (at 157.48 101.6062 0)
       (effects (font (size 1.27 1.27)) (justify left))
     )
@@
       (effects (font (size 1.27 1.27)) hide)
     )
-    (property "Value" "+5V" (id 1) (at 157.48 129.5399 0)
-      (effects (font (size 1.27 1.27)) (justify left))
-    )
+    (property "Value" "+5V" (id 1) (at 154.94 125.73 0))
     (property "Footprint" "" (id 2) (at 154.94 130.81 0)
       (effects (font (size 1.27 1.27)) hide)
@@
   (symbol (lib_id "Device:C_Polarized_Small") (at 229.87 50.8 0) (unit 1)
     (in_bom yes) (on_board yes) (fields_autoplaced)
-    (property "Reference" "C15" (id 0) (at 233.172 48.9838 0)
-      (effects (font (size 1.27 1.27)) (justify left))
-    )
-    (property "Value" "470uF 20 V" (id 1) (at 233.172 51.5238 0)
+    (property "Reference" "C15" (id 0) (at 232.41 48.9838 0)
+      (effects (font (size 1.27 1.27)) (justify left))
+    )
+    (property "Value" "470uF 20 V" (id 1) (at 232.41 51.5238 0)
       (effects (font (size 1.27 1.27)) (justify left))
     )
@@
   (symbol (lib_id "Device:C_Polarized_Small") (at 140.97 52.07 0) (unit 1)
     (in_bom yes) (on_board yes) (fields_autoplaced)
-    (property "Reference" "C17" (id 0) (at 138.684 50.2538 0)
+    (property "Reference" "C17" (id 0) (at 138.43 50.2538 0)
       (effects (font (size 1.27 1.27)) (justify right))
     )
-    (property "Value" "470uF 20 V" (id 1) (at 138.684 52.7938 0)
+    (property "Value" "470uF 20 V" (id 1) (at 138.43 52.7938 0)
       (effects (font (size 1.27 1.27)) (justify right))
     )
@@
   (symbol (lib_id "Device:C_Polarized_Small") (at 246.38 100.33 0) (unit 1)
     (in_bom yes) (on_board yes) (fields_autoplaced)
-    (property "Reference" "C26" (id 0) (at 249.682 98.5138 0)
-      (effects (font (size 1.27 1.27)) (justify left))
-    )
-    (property "Value" "470uF 20 V" (id 1) (at 249.682 101.0538 0)
+    (property "Reference" "C26" (id 0) (at 248.92 98.5138 0)
+      (effects (font (size 1.27 1.27)) (justify left))
+    )
+    (property "Value" "470uF 20 V" (id 1) (at 248.92 101.0538 0)
       (effects (font (size 1.27 1.27)) (justify left))
     )
@@
   (symbol (lib_id "Device:C_Polarized_Small") (at 229.87 100.33 0) (unit 1)
     (in_bom yes) (on_board yes) (fields_autoplaced)
-    (property "Reference" "C25" (id 0) (at 233.172 98.5138 0)
-      (effects (font (size 1.27 1.27)) (justify left))
-    )
-    (property "Value" "470uF 20 V" (id 1) (at 233.172 101.0538 0)
+    (property "Reference" "C25" (id 0) (at 232.41 98.5138 0)
+      (effects (font (size 1.27 1.27)) (justify left))
+    )
+    (property "Value" "470uF 20 V" (id 1) (at 232.41 101.0538 0)
       (effects (font (size 1.27 1.27)) (justify left))
     )
@@
       (effects (font (size 1.27 1.27)) hide)
     )
-    (property "Value" "+3V3" (id 1) (at 170.18 129.5399 0)
-      (effects (font (size 1.27 1.27)) (justify left))
-    )
+    (property "Value" "+3V3" (id 1) (at 167.64 125.73 0))
     (property "Footprint" "" (id 2) (at 167.64 130.81 0)
       (effects (font (size 1.27 1.27)) hide)
@@
   (symbol (lib_id "Device:C_Small") (at 200.66 50.8 0) (unit 1)
     (in_bom yes) (on_board yes) (fields_autoplaced)
-    (property "Reference" "C13" (id 0) (at 203.454 49.5362 0)
-      (effects (font (size 1.27 1.27)) (justify left))
-    )
-    (property "Value" "10uF 16 V" (id 1) (at 203.454 52.0762 0)
+    (property "Reference" "C13" (id 0) (at 203.2 49.5362 0)
+      (effects (font (size 1.27 1.27)) (justify left))
+    )
+    (property "Value" "10uF 16 V" (id 1) (at 203.2 52.0762 0)
       (effects (font (size 1.27 1.27)) (justify left))
     )
@@
       (effects (font (size 1.27 1.27)) hide)
     )
-    (property "Value" "NetTie_2" (id 1) (at 34.29 87.63 0)
+    (property "Value" "NetTie" (id 1) (at 34.29 87.63 0)
       (effects (font (size 1.27 1.27)) hide)
     )
@@
   (symbol (lib_id "Device:C_Small") (at 215.9 100.33 0) (unit 1)
     (in_bom yes) (on_board yes) (fields_autoplaced)
-    (property "Reference" "C24" (id 0) (at 218.948 99.0662 0)
-      (effects (font (size 1.27 1.27)) (justify left))
-    )
-    (property "Value" "22uF 16 V" (id 1) (at 218.948 101.6062 0)
+    (property "Reference" "C24" (id 0) (at 218.44 99.0662 0)
+      (effects (font (size 1.27 1.27)) (justify left))
+    )
+    (property "Value" "22uF 16 V" (id 1) (at 218.44 101.6062 0)
       (effects (font (size 1.27 1.27)) (justify left))
     )
@@
   (symbol (lib_id "Device:C_Small") (at 154.94 50.8 0) (unit 1)
     (in_bom yes) (on_board yes) (fields_autoplaced)
-    (property "Reference" "C11" (id 0) (at 158.496 49.5362 0)
-      (effects (font (size 1.27 1.27)) (justify left))
-    )
-    (property "Value" "10uF 16 V" (id 1) (at 158.496 52.0762 0)
+    (property "Reference" "C11" (id 0) (at 157.48 49.5362 0)
+      (effects (font (size 1.27 1.27)) (justify left))
+    )
+    (property "Value" "10uF 16 V" (id 1) (at 157.48 52.0762 0)
       (effects (font (size 1.27 1.27)) (justify left))
     )
@@
   (symbol (lib_id "Device:C_Small") (at 215.9 50.8 0) (unit 1)
     (in_bom yes) (on_board yes) (fields_autoplaced)
-    (property "Reference" "C14" (id 0) (at 218.948 49.5362 0)
-      (effects (font (size 1.27 1.27)) (justify left))
-    )
-    (property "Value" "22uF 16 V" (id 1) (at 218.948 52.0762 0)
+    (property "Reference" "C14" (id 0) (at 218.44 49.5362 0)
+      (effects (font (size 1.27 1.27)) (justify left))
+    )
+    (property "Value" "22uF 16 V" (id 1) (at 218.44 52.0762 0)
       (effects (font (size 1.27 1.27)) (justify left))
     )
@@
       (effects (font (size 1.27 1.27)) hide)
     )
-    (property "Value" "+12V" (id 1) (at 143.51 129.5399 0)
-      (effects (font (size 1.27 1.27)) (justify left))
-    )
+    (property "Value" "+12V" (id 1) (at 140.97 125.73 0))
     (property "Footprint" "" (id 2) (at 140.97 130.81 0)
       (effects (font (size 1.27 1.27)) hide)
@@
   (symbol (lib_id "Device:C_Small") (at 200.66 100.33 0) (unit 1)
     (in_bom yes) (on_board yes) (fields_autoplaced)
-    (property "Reference" "C23" (id 0) (at 203.454 99.0662 0)
-      (effects (font (size 1.27 1.27)) (justify left))
-    )
-    (property "Value" "10uF 16 V" (id 1) (at 203.454 101.6062 0)
-      (effects (font (size 1.27 1.27)) (justify left))
-    )
+    (property "Reference" "C23" (id 0) (at 203.2 99.0662 0)
+      (effects (font (size 1.27 1.27)) (justify left))
+    )
+    (property "Value" "10uF 16 V" (id 1) (at 203.2 101.6062 0)
+      (effects (font (size 1.27 1.27)) (justify left))
+    )
