File: CIB_Main_PCB - Mimic Octopus/CIB_Main_PCB.kicad_sch (KiCad schematic)
At the start: 24 parts, among them J10 External IO, J15 DUT PSU, J16 CIB Power

Commit message: message
Parts:
- J15: value DUT PSU -> DUT Power Out
- J16: footprint 1864053 -> Component Search Engine:Pluggable Terminal Blocks SDC 2,5 4-PV-5,0 0-ZB
Connections:
- net +VDC: now also J16.3; no longer J16.2
- net -VDC: now also J16.2; no longer J16.3
- net DUT Power 1 +VE: now also J15.5; no longer J15.2
- net DUT Power 1 -VE: now also J15.2; no longer J15.5
- net DUT Power 2 +VE: now also J15.11; no longer J15.8
- net DUT Power 2 -VE: now also J15.8; no longer J15.11

Commit message: added changes
Parts:
- J1: renamed from J10; footprint Component Search Engine:Pluggable Terminal Blocks SDDC 1,5 14-PV-3,5 -> Component Search Engine:Pluggable Terminal Blocks SDDC 1.5mm pitch 28 Pin
- J2: renamed from J15; footprint Component Search Engine:Pluggable Terminal Blocks SDC 2,5 12-PV-5,0 0-ZB -> Component Search Engine:Pluggable Terminal Blocks SDC 2.5mm pitch 12 Pin
- J3: renamed from J16; footprint Component Search Engine:Pluggable Terminal Blocks SDC 2,5 4-PV-5,0 0-ZB -> Component Search Engine:Pluggable Terminal Blocks SDC 2.5mm pitch 4 Pin
- renumbered H6 to H10, H12 to H11, H13 to H12, H17 to H13, H20 to H14, H7 to H15, H8 to H16, H9 to H17, H14 to H18, H15 to H19, H18 to H20, H10 to H4, H11 to H5, H16 to H6, H19 to H7, H4 to H8, H5 to H9

Commit message: changes
Connections:
- net -VDC is gone; now on net GND: J3.2, J3.4
Changed lines of the file:
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@@
     (pin "1")
   )
-  (symbol (lib_id "power:-VDC") (at 177.8 132.08 180) (unit 1)
-    (in_bom yes) (on_board yes)
-    (property "Reference" "#PWR010" (id 0) (at 177.8 129.54 0)
-      (effects (font (size 1.27 1.27)) hide)
-    )
-    (property "Value" "-VDC" (id 1) (at 177.8 139.7 0))
+  (symbol (lib_id "power:GND") (at 177.8 132.08 0) (unit 1)
+    (in_bom yes) (on_board yes) (fields_autoplaced)
+    (property "Reference" "#PWR0104" (id 0) (at 177.8 138.43 0)
+      (effects (font (size 1.27 1.27)) hide)
+    )
+    (property "Value" "GND" (id 1) (at 177.8 137.16 0))
     (property "Footprint" "" (id 2) (at 177.8 132.08 0)
       (effects (font (size 1.27 1.27)) hide)
@@
       (reference "#PWR09") (unit 1) (value "+VDC") (footprint "")
     )
-    (path "/5633b50d-bc60-4c4e-a38b-4e23d1469a07"
-      (reference "#PWR010") (unit 1) (value "-VDC") (footprint "")
-    )
     (path "/f846a415-d0bf-4a59-8df3-19661627a82e"
       (reference "#PWR011") (unit 1) (value "GND") (footprint "")
@@
       (reference "#PWR0103") (unit 1) (value "GND") (footprint "")
     )
-    (path "/d19b6226-223c-4818-843d-8965d7e15487/39f7d7ab-8b1f-4432-b528-9727e19eb3d3"
-      (reference "#PWR0104") (unit 1) (value "-VDC") (footprint "")
+    (path "/553c14d0-1540-4670-aea9-b15f19caad2e"
+      (reference "#PWR0104") (unit 1) (value "GND") (footprint "")
     )
     (path "/d19b6226-223c-4818-843d-8965d7e15487/fda2c003-b2fe-4dcd-b571-06fda0e7b682"
@@
       (reference "#PWR0378") (unit 1) (value "~") (footprint "")
     )
+    (path "/d19b6226-223c-4818-843d-8965d7e15487/e822e928-2879-4930-a98b-5cbfa46bfeb9"
+      (reference "#PWR0379") (unit 1) (value "GND") (footprint "")
+    )
     (path "/bf197791-f0c1-45bf-ae92-0afefa911606/67281890-be1c-4753-8cf4-8737fc2a3e55"

Commit message: V0.1 PCB to be sent out
Parts:
- removed J3: CIB Power, Component Search Engine:Pluggable Terminal Blocks SDC 2.5mm pitch 4 Pin, symbol Component Search Engine:Pluggable Terminal Blocks SDC 2,5/ 4-PV-5,0 0-ZB
- added H22, H23, H24, H25, H26, H27: M4, MountingHole:MountingHole_4.3mm_M4_DIN965_Pad, symbol Mechanical:MountingHole_Pad
- added J16: External IO 2, Component Search Engine:Pluggable Terminal Blocks SDDC 1.5mm pitch 32 Pin, symbol _SKDD Connectors:Pluggable Terminal Blocks SDDC 1.5mm pitch 32 Pin
- J1: value External IO -> External IO 1
Connections:
- net Misc Relays/RAG AMBER is gone; now on net INTERLOCK LOOP: J1.27
- net Misc Relays/RAG GREEN is gone; now on net TEST START: J1.28
- net Misc Relays/RAG RED is gone; now on net DOOR CLOSED: J1.26
- net +12V: now also J16.1, J16.17
- net +3V3: now also J16.19, J16.3
- net +5V: now also J1.25, J16.18, J16.2; no longer J1.11
- net DIO 1: now also J1.4; no longer J1.7
- net DIO 2: now also J1.5; no longer J1.6
- net DIO 3: now also J1.6; no longer J1.5
- net DOOR CLOSED: no longer J1.14
- net GND: now also J1.11, H22.1, H23.1, H24.1, H25.1, H26.1, H27.1, J16.20, J16.22, J16.4, J16.6; no longer J1.25
- net HV PSU: now also J1.18; no longer J1.4
- net INTERLOCK LOOP: no longer J1.13
- net Misc Relays/External Relay 1: now also J1.24; no longer J1.23
- net Misc Relays/External Relay 2: now also J1.23; no longer J1.22
- net Misc Relays/External Relay 3: now also J1.22; no longer J1.21
- net Misc Relays/External Relay 4: now also J1.21; no longer J1.20
- net Misc Relays/External Relay 5: now also J1.20; no longer J1.19
- net Misc Relays/External Relay 6: now also J1.19; no longer J1.18
- net TEST START: no longer J1.12
- net DIO 7: now reaches J1.10
- net DIO 5: now reaches J1.8
- net DIO 6: now reaches J1.9
- new net AIO1: J16.21
- new net AIO2: J16.5
- new net DIO 4: J1.7
- new net RAG A: J1.13
- new net RAG G: J1.14
- new net RAG R: J1.12
Other:
- sheet Cross Point Matrix ports: added Clock, Din, Dout, Latch; removed SCL, SDA
- sheet MicroControler Interface ports: added AIN14, AIN15, Clock, Din, Dout, Latch; removed none
- sheet Misc Relays ports: added Clock, DIN, DOUT, Latch; removed SCL 5V, SDA 5V
- sheet Power Supply ports: added CIB 5V monitor; removed none
- moved on the sheet: J1, J2

Commit message: BoM
Parts:
- H1, H10, H11, H12, H13, H14, H15, H16, H17, H18, H19, H2, H20, H21, H22, H23, H24, H25, H26, H27, H3, H4, H5, H6, H7, H8, H9: dnp (none) -> dnp
- J1: Height (none) -> 16; Manufacturer_Part_Number 1848765 -> (none); Mouser # (none) -> 651-1848765; Mouser Part Number 651-1848765 -> (none)
- J16: Height (none) -> 16; Manufacturer (none) -> Phoenix Contact; Manufacturer # (none) -> 1848781; Manufacturer_Name Phoenix Contact -> (none); Manufacturer_Part_Number 1848781 -> (none); Mouser # (none) -> 651-1848781; Mouser Part Number 651-1848781 -> (none)
- J2: Mouser # (none) -> 651-1864134; Mouser Part Number 651-1864134 -> (none)

Commit message: changes
Parts:
- removed J2: DUT Power Out, Component Search Engine:Pluggable Terminal Blocks SDC 2.5mm pitch 12 Pin, symbol Component Search Engine:Pluggable Terminal Blocks SDC 2,5/12-PV-5,0 0-ZB
Other:
- sheet Misc Relays ports: added none; removed DUT Power 1 +VE, DUT Power 1 -VE, DUT Power 2 +VE, DUT Power 2 -VE
