File: CIB_Main_PCB - Mimic Octopus/Cross Point Matix Ch1-4.kicad_sch (KiCad schematic)
At the start: 7 parts, among them U10 ULN2803A, U12 ULN2803A, U5 MCP23017_SO

Commit message: added changes
Parts:
- removed U10, U12: ULN2803A, Package_DIP:DIP-18_W7.62mm_LongPads, symbol Transistor_Array:ULN2803A
- removed U5: MCP23017_SO, Package_SO:SOIC-28W_7.5x17.9mm_P1.27mm, symbol Interface_Expansion:MCP23017_SO
- added U10, U12: 74HC595, Package_DIP:DIP-16_W7.62mm_LongPads, symbol 74xx:74HC595
- added U11, U15: ULN2803A, Package_DIP:DIP-18_W7.62mm_LongPads, symbol Transistor_Array:ULN2803A
- renumbered C28 to C32, C29 to C33, C30 to C34, C31 to C35
Connections:
- net +12V: now also U11.10 (COM), U15.10 (COM)
- net +5V: now also U10.10 (~{SRCLR}), U10.16 (VCC), U12.10 (~{SRCLR}), U12.16 (VCC)
- net Cross Point Matrix 8 Relays (High Current) a/Relay 1: now also U11.18 (O1)
- net Cross Point Matrix 8 Relays (High Current) a/Relay 2: now also U11.17 (O2)
- net Cross Point Matrix 8 Relays (High Current) a/Relay 3: now also U11.16 (O3)
- net Cross Point Matrix 8 Relays (High Current) a/Relay 4: now also U11.15 (O4)
- net Cross Point Matrix 8 Relays (High Current) a/Relay 5: now also U11.14 (O5)
- net Cross Point Matrix 8 Relays (High Current) a/Relay 6: now also U11.13 (O6)
- net Cross Point Matrix 8 Relays (High Current) a/Relay 7: now also U11.12 (O7)
- net Cross Point Matrix 8 Relays (High Current) a/Relay 8: now also U11.11 (O8)
- net Cross Point Matrix 8 Relays (High Current) b/Relay 1: now also U15.18 (O1)
- net Cross Point Matrix 8 Relays (High Current) b/Relay 2: now also U15.17 (O2)
- net Cross Point Matrix 8 Relays (High Current) b/Relay 3: now also U15.16 (O3)
- net Cross Point Matrix 8 Relays (High Current) b/Relay 4: now also U15.15 (O4)
- net Cross Point Matrix 8 Relays (High Current) b/Relay 5: now also U15.14 (O5)
- net Cross Point Matrix 8 Relays (High Current) b/Relay 6: now also U15.13 (O6)
- net Cross Point Matrix 8 Relays (High Current) b/Relay 7: now also U15.12 (O7)
- net Cross Point Matrix 8 Relays (High Current) b/Relay 8: now also U15.11 (O8)
- net GND: now also U10.13 (~{OE}), U10.8 (GND), U11.9 (GND), U12.13 (~{OE}), U12.8 (GND), U15.9 (GND)
- new net: U12.1 (QB), U15.7 (I7)
- new net: U10.9 (QH'), U12.14 (SER)
- new net: U12.15 (QA), U15.8 (I8)
- new net: U12.2 (QC), U15.6 (I6)
- new net: U12.3 (QD), U15.5 (I5)
- new net: U12.4 (QE), U15.4 (I4)
- new net: U12.5 (QF), U15.3 (I3)
- new net: U12.6 (QG), U15.2 (I2)
- new net: U12.7 (QH), U15.1 (I1)
- new net: U10.7 (QH), U11.1 (I1)
- new net: U10.6 (QG), U11.2 (I2)
- new net: U10.5 (QF), U11.3 (I3)
- new net: U10.4 (QE), U11.4 (I4)
- new net: U10.3 (QD), U11.5 (I5)
- new net: U10.2 (QC), U11.6 (I6)
- new net: U10.1 (QB), U11.7 (I7)
- new net: U10.15 (QA), U11.8 (I8)
- new net Clock: U10.11 (SRCLK), U12.11 (SRCLK)
- new net DIN: U10.14 (SER)
- new net DOUT: U12.9 (QH')
- new net Latch: U10.12 (RCLK), U12.12 (RCLK)

Commit message: changes
Changed lines of the file:
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@@
     (effects (font (size 1.27 1.27)) (justify left))
   )
-  (hierarchical_label "I{slash}O Ch2 High" (shape input) (at 177.8 77.47 180)
+  (hierarchical_label "I{slash}O Ch2 High" (shape input) (at 177.8 72.39 180)
     (effects (font (size 1.27 1.27)) (justify right))
   )
-  (hierarchical_label "I{slash}O Ch2 Low" (shape input) (at 177.8 80.01 180)
+  (hierarchical_label "I{slash}O Ch2 Low" (shape input) (at 177.8 74.93 180)
     (effects (font (size 1.27 1.27)) (justify right))
   )
@@
     (effects (font (size 1.27 1.27)) (justify left))
   )
-  (hierarchical_label "I{slash}O Ch4 High" (shape input) (at 177.8 134.62 180)
+  (hierarchical_label "I{slash}O Ch4 High" (shape input) (at 177.8 129.54 180)
     (effects (font (size 1.27 1.27)) (justify right))
   )
@@
     (effects (font (size 1.27 1.27)) (justify left))
   )
-  (hierarchical_label "I{slash}O Ch4 Low" (shape input) (at 177.8 137.16 180)
+  (hierarchical_label "I{slash}O Ch4 Low" (shape input) (at 177.8 132.08 180)
     (effects (font (size 1.27 1.27)) (justify right))
   )
@@
     (effects (font (size 1.27 1.27)) (justify left))
   )
-  (hierarchical_label "I{slash}O Ch3 Low" (shape input) (at 177.8 132.08 180)
+  (hierarchical_label "I{slash}O Ch3 Low" (shape input) (at 177.8 137.16 180)
     (effects (font (size 1.27 1.27)) (justify right))
   )
@@
     (effects (font (size 1.27 1.27)) (justify left))
   )
-  (hierarchical_label "I{slash}O Ch1 Low" (shape input) (at 177.8 74.93 180)
+  (hierarchical_label "I{slash}O Ch1 Low" (shape input) (at 177.8 80.01 180)
     (effects (font (size 1.27 1.27)) (justify right))
   )
@@
     (effects (font (size 1.27 1.27)) (justify left))
   )
-  (hierarchical_label "I{slash}O Ch1 High" (shape input) (at 177.8 72.39 180)
+  (hierarchical_label "I{slash}O Ch1 High" (shape input) (at 177.8 77.47 180)
     (effects (font (size 1.27 1.27)) (justify right))
   )
@@
     (effects (font (size 1.27 1.27)) (justify right))
   )
-  (hierarchical_label "I{slash}O Ch3 High" (shape input) (at 177.8 129.54 180)
+  (hierarchical_label "I{slash}O Ch3 High" (shape input) (at 177.8 134.62 180)
     (effects (font (size 1.27 1.27)) (justify right))
   )

Commit message: BoM
Parts:
- C32, C34: Height (none) -> 2
- C33, C35: DigiKey # 732-7642-1-ND -> 1276-3048-1-ND; DigiKey Price/Stock https://www.digikey.co.uk/en/products/detail/w%C3%BCrth-ele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 -> https://www.digikey.co.uk/en/products/detail/samsung-electr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; Height (none) -> 2; Manufacturer Würth Elektronik -> Samsung Electro-Mechanics; Manufacturer # 885012108018 -> CL31A226KOHNNNE
- U10, U12: Height (none) -> 5
- U11, U15: Height (none) -> 5; Mouser # (none) -> 511-ULN2803A; Mouser Part Number 511-ULN2803A -> (none)
Changed lines of the file:
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@@
+      (effects (font (size 1.27 1.27)) hide)
+    )
+    (property "Height" "5" (id 4) (at 113.03 97.79 0)
       (effects (font (size 1.27 1.27)) hide)
     )
@@
       (effects (font (size 1.27 1.27)) hide)
     )
-    (property "Datasheet" "https://www.we-online.com/katalog/datasheet/885012108018.pdf" (id 3) (at 46.99 78.74 0)
-      (effects (font (size 1.27 1.27)) hide)
-    )
-    (property "Manufacturer #" "885012108018" (id 4) (at 46.99 78.74 0)
-      (effects (font (size 1.27 1.27)) hide)
-    )
-    (property "DigiKey #" "732-7642-1-ND" (id 5) (at 46.99 78.74 0)
-      (effects (font (size 1.27 1.27)) hide)
-    )
-    (property "Manufacturer" "Würth Elektronik" (id 6) (at 46.99 78.74 0)
+    (property "Datasheet" "https://media.digikey.com/pdf/Data%20Sheets/Samsung%20PDFs/CL31B106KOHNNNE_Spec.pdf" (id 3) (at 46.99 78.74 0)
+      (effects (font (size 1.27 1.27)) hide)
+    )
+    (property "Manufacturer #" "CL31A226KOHNNNE" (id 4) (at 46.99 78.74 0)
+      (effects (font (size 1.27 1.27)) hide)
+    )
+    (property "DigiKey #" "1276-3048-1-ND" (id 5) (at 46.99 78.74 0)
+      (effects (font (size 1.27 1.27)) hide)
+    )
+    (property "Manufacturer" "Samsung Electro-Mechanics" (id 6) (at 46.99 78.74 0)
       (effects (font (size 1.27 1.27)) hide)
     )
@@
       (effects (font (size 1.27 1.27)) hide)
     )
-    (property "DigiKey Price/Stock" "https://www.digikey.co.uk/en/products/detail/w%C3%BCrth-elektronik/885012108018/5453497?s=N4IgTCBcDaIOwGYwFo4DYAsKCMyByAIiALoC%2BQA" (id 8) (at 46.99 78.74 0)
+    (property "DigiKey Price/Stock" "https://www.digikey.co.uk/en/products/detail/samsung-electro-mechanics/CL31A226KOHNNNE/3888706" (id 8) (at 46.99 78.74 0)
+      (effects (font (size 1.27 1.27)) hide)
+    )
+    (property "Height" "2" (id 9) (at 46.99 78.74 0)
       (effects (font (size 1.27 1.27)) hide)
     )
@@
       (effects (font (size 1.27 1.27)) hide)
     )
+    (property "Height" "2" (id 9) (at 31.75 78.74 0)
+      (effects (font (size 1.27 1.27)) hide)
+    )
     (pin "1")
     (pin "2")
@@
       (effects (font (size 1.27 1.27)) hide)
     )
-    (property "Datasheet" "https://www.we-online.com/katalog/datasheet/885012108018.pdf" (id 3) (at 46.99 48.26 0)
-      (effects (font (size 1.27 1.27)) hide)
-    )
-    (property "Manufacturer #" "885012108018" (id 4) (at 46.99 48.26 0)
-      (effects (font (size 1.27 1.27)) hide)
-    )
-    (property "DigiKey #" "732-7642-1-ND" (id 5) (at 46.99 48.26 0)
-      (effects (font (size 1.27 1.27)) hide)
-    )
-    (property "Manufacturer" "Würth Elektronik" (id 6) (at 46.99 48.26 0)
+    (property "Datasheet" "https://media.digikey.com/pdf/Data%20Sheets/Samsung%20PDFs/CL31B106KOHNNNE_Spec.pdf" (id 3) (at 46.99 48.26 0)
+      (effects (font (size 1.27 1.27)) hide)
+    )
+    (property "Manufacturer #" "CL31A226KOHNNNE" (id 4) (at 46.99 48.26 0)
+      (effects (font (size 1.27 1.27)) hide)
+    )
+    (property "DigiKey #" "1276-3048-1-ND" (id 5) (at 46.99 48.26 0)
+      (effects (font (size 1.27 1.27)) hide)
+    )
+    (property "Manufacturer" "Samsung Electro-Mechanics" (id 6) (at 46.99 48.26 0)
       (effects (font (size 1.27 1.27)) hide)
     )
@@
       (effects (font (size 1.27 1.27)) hide)
     )
-    (property "DigiKey Price/Stock" "https://www.digikey.co.uk/en/products/detail/w%C3%BCrth-elektronik/885012108018/5453497?s=N4IgTCBcDaIOwGYwFo4DYAsKCMyByAIiALoC%2BQA" (id 8) (at 46.99 48.26 0)
+    (property "DigiKey Price/Stock" "https://www.digikey.co.uk/en/products/detail/samsung-electro-mechanics/CL31A226KOHNNNE/3888706" (id 8) (at 46.99 48.26 0)
+      (effects (font (size 1.27 1.27)) hide)
+    )
+    (property "Height" "2" (id 9) (at 46.99 48.26 0)
       (effects (font (size 1.27 1.27)) hide)
     )
@@
       (effects (font (size 1.27 1.27)) hide)
     )
-    (property "Mouser #" "" (id 8) (at 153.67 53.34 0)
-      (effects (font (size 1.27 1.27)) hide)
-    )
-    (property "Mouser Part Number" "511-ULN2803A" (id 9) (at 153.67 53.34 0)
+    (property "Mouser #" "511-ULN2803A" (id 8) (at 153.67 53.34 0)
+      (effects (font (size 1.27 1.27)) hide)
+    )
+    (property "Mouser Part Number" "" (id 9) (at 153.67 53.34 0)
+      (effects (font (size 1.27 1.27)) hide)
+    )
+    (property "Height" "5" (id 10) (at 153.67 53.34 0)
       (effects (font (size 1.27 1.27)) hide)
     )
@@
       (effects (font (size 1.27 1.27)) hide)
     )
+    (property "Height" "5" (id 4) (at 113.03 40.64 0)
+      (effects (font (size 1.27 1.27)) hide)
+    )
     (pin "1")
     (pin "10")
@@
       (effects (font (size 1.27 1.27)) hide)
     )
-    (property "Mouser #" "" (id 8) (at 153.67 110.49 0)
-      (effects (font (size 1.27 1.27)) hide)
-    )
-    (property "Mouser Part Number" "511-ULN2803A" (id 9) (at 153.67 110.49 0)
+    (property "Mouser #" "511-ULN2803A" (id 8) (at 153.67 110.49 0)
+      (effects (font (size 1.27 1.27)) hide)
+    )
+    (property "Mouser Part Number" "" (id 9) (at 153.67 110.49 0)
+      (effects (font (size 1.27 1.27)) hide)
+    )
+    (property "Height" "5" (id 10) (at 153.67 110.49 0)
       (effects (font (size 1.27 1.27)) hide)
     )
@@
       (effects (font (size 1.27 1.27)) hide)
     )
+    (property "Height" "2" (id 9) (at 31.75 48.26 0)
+      (effects (font (size 1.27 1.27)) hide)
+    )
