File: CIB_Main_PCB - Mimic Octopus/Cross Point Matix Ch17-24.kicad_sch (KiCad schematic)
At the start: 7 parts, among them U23 MCP23017_SO, U26 MCP23018, U28 MCP23018

Commit message: added changes
Parts:
- removed U23: MCP23017_SO, Package_SO:SOIC-28W_7.5x17.9mm_P1.27mm, symbol Interface_Expansion:MCP23017_SO
- removed U26: MCP23018, Package_DIP:DIP-18_W7.62mm_LongPads, symbol Transistor_Array:ULN2803A
- added U26, U29: 74HC595, Package_DIP:DIP-16_W7.62mm_LongPads, symbol 74xx:74HC595
- added U30: ULN2803A, Package_DIP:DIP-18_W7.62mm_LongPads, symbol Transistor_Array:ULN2803A
- U28: value MCP23018 -> ULN2803A
- renumbered C48 to C52, C49 to C53, C50 to C54, C51 to C55
Connections:
- net +12V: now also U30.10 (COM)
- net +5V: now also U26.10 (~{SRCLR}), U26.16 (VCC), U29.10 (~{SRCLR}), U29.16 (VCC)
- net Cross Point Matrix 8 Relays (Low Current) b/Relay 1: no longer U28.15 (O4)
- net Cross Point Matrix 8 Relays (Low Current) b/Relay 2: no longer U28.16 (O3)
- net Cross Point Matrix 8 Relays (Low Current) b/Relay 3: no longer U28.17 (O2)
- net Cross Point Matrix 8 Relays (Low Current) b/Relay 4: no longer U28.18 (O1)
- net Cross Point Matrix 8 Relays (Low Current) b/Relay 5: no longer U28.14 (O5)
- net Cross Point Matrix 8 Relays (Low Current) b/Relay 6: no longer U28.13 (O6)
- net Cross Point Matrix 8 Relays (Low Current) b/Relay 7: no longer U28.12 (O7)
- net Cross Point Matrix 8 Relays (Low Current) b/Relay 8: no longer U28.11 (O8)
- net GND: now also U26.13 (~{OE}), U26.8 (GND), U29.13 (~{OE}), U29.8 (GND), U30.9 (GND)
- net at U28.8 (I8): now also U26.15 (QA)
- net at U28.7 (I7): now also U26.1 (QB)
- net at U28.6 (I6): now also U26.2 (QC)
- net at U28.5 (I5): now also U26.3 (QD)
- net at U28.4 (I4): now also U26.4 (QE)
- net at U28.3 (I3): now also U26.5 (QF)
- net at U28.2 (I2): now also U26.6 (QG)
- net at U28.1 (I1): now also U26.7 (QH)
- new net: U29.7 (QH), U30.1 (I1)
- new net: U29.6 (QG), U30.2 (I2)
- new net: U29.5 (QF), U30.3 (I3)
- new net: U29.4 (QE), U30.4 (I4)
- new net: U29.3 (QD), U30.5 (I5)
- new net: U29.2 (QC), U30.6 (I6)
- new net: U29.1 (QB), U30.7 (I7)
- new net: U29.15 (QA), U30.8 (I8)
- new net: U26.9 (QH'), U29.14 (SER)
- new net Clock: U26.11 (SRCLK), U29.11 (SRCLK)
- new net DIN: U26.14 (SER)
- new net DOUT: U29.9 (QH')
- new net Latch: U26.12 (RCLK), U29.12 (RCLK)

Commit message: V0.1 PCB to be sent out
Connections:
- net Cross Point Matrix 8 Relays (Low Current) a/Relay 1: now also U28.14 (O5)
- net Cross Point Matrix 8 Relays (Low Current) a/Relay 2: now also U28.13 (O6)
- net Cross Point Matrix 8 Relays (Low Current) a/Relay 3: now also U28.12 (O7)
- net Cross Point Matrix 8 Relays (Low Current) a/Relay 4: now also U28.11 (O8)
- net Cross Point Matrix 8 Relays (Low Current) a/Relay 5: now also U28.15 (O4)
- net Cross Point Matrix 8 Relays (Low Current) a/Relay 6: now also U28.16 (O3)
- net Cross Point Matrix 8 Relays (Low Current) a/Relay 7: now also U28.17 (O2)
- net Cross Point Matrix 8 Relays (Low Current) a/Relay 8: now also U28.18 (O1)
- net Cross Point Matrix 8 Relays (Low Current) b/Relay 1: now also U30.14 (O5)
- net Cross Point Matrix 8 Relays (Low Current) b/Relay 2: now also U30.13 (O6)
- net Cross Point Matrix 8 Relays (Low Current) b/Relay 3: now also U30.12 (O7)
- net Cross Point Matrix 8 Relays (Low Current) b/Relay 4: now also U30.11 (O8)
- net Cross Point Matrix 8 Relays (Low Current) b/Relay 5: now also U30.15 (O4)
- net Cross Point Matrix 8 Relays (Low Current) b/Relay 6: now also U30.16 (O3)
- net Cross Point Matrix 8 Relays (Low Current) b/Relay 7: now also U30.17 (O2)
- net Cross Point Matrix 8 Relays (Low Current) b/Relay 8: now also U30.18 (O1)

Commit message: BoM
Parts:
- C52, C54: Height (none) -> 2
- C53, C55: DigiKey # 732-7642-1-ND -> 1276-3048-1-ND; DigiKey Price/Stock https://www.digikey.co.uk/en/products/detail/w%C3%BCrth-ele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 -> https://www.digikey.co.uk/en/products/detail/samsung-electr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; Height (none) -> 2; Manufacturer Würth Elektronik -> Samsung Electro-Mechanics; Manufacturer # 885012108018 -> CL31A226KOHNNNE
- U26, U29: Height (none) -> 5
- U28, U30: Height (none) -> 5; Mouser # (none) -> 511-ULN2803A; Mouser Part Number 511-ULN2803A -> (none)
Changed lines of the file:
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@@
       (effects (font (size 1.27 1.27)) hide)
     )
-    (property "Datasheet" "https://www.we-online.com/katalog/datasheet/885012108018.pdf" (id 3) (at 48.26 53.34 0)
-      (effects (font (size 1.27 1.27)) hide)
-    )
-    (property "Manufacturer #" "885012108018" (id 4) (at 48.26 53.34 0)
-      (effects (font (size 1.27 1.27)) hide)
-    )
-    (property "DigiKey #" "732-7642-1-ND" (id 5) (at 48.26 53.34 0)
-      (effects (font (size 1.27 1.27)) hide)
-    )
-    (property "Manufacturer" "Würth Elektronik" (id 6) (at 48.26 53.34 0)
+    (property "Datasheet" "https://media.digikey.com/pdf/Data%20Sheets/Samsung%20PDFs/CL31B106KOHNNNE_Spec.pdf" (id 3) (at 48.26 53.34 0)
+      (effects (font (size 1.27 1.27)) hide)
+    )
+    (property "Manufacturer #" "CL31A226KOHNNNE" (id 4) (at 48.26 53.34 0)
+      (effects (font (size 1.27 1.27)) hide)
+    )
+    (property "DigiKey #" "1276-3048-1-ND" (id 5) (at 48.26 53.34 0)
+      (effects (font (size 1.27 1.27)) hide)
+    )
+    (property "Manufacturer" "Samsung Electro-Mechanics" (id 6) (at 48.26 53.34 0)
       (effects (font (size 1.27 1.27)) hide)
     )
@@
       (effects (font (size 1.27 1.27)) hide)
     )
-    (property "DigiKey Price/Stock" "https://www.digikey.co.uk/en/products/detail/w%C3%BCrth-elektronik/885012108018/5453497?s=N4IgTCBcDaIOwGYwFo4DYAsKCMyByAIiALoC%2BQA" (id 8) (at 48.26 53.34 0)
+    (property "DigiKey Price/Stock" "https://www.digikey.co.uk/en/products/detail/samsung-electro-mechanics/CL31A226KOHNNNE/3888706" (id 8) (at 48.26 53.34 0)
+      (effects (font (size 1.27 1.27)) hide)
+    )
+    (property "Height" "2" (id 9) (at 48.26 53.34 0)
       (effects (font (size 1.27 1.27)) hide)
     )
@@
       (effects (font (size 1.27 1.27)) hide)
     )
+    (property "Height" "2" (id 9) (at 33.02 83.82 0)
+      (effects (font (size 1.27 1.27)) hide)
+    )
     (pin "1")
     (pin "2")
@@
     )
     (property "DigiKey Price/Stock" "https://www.digikey.co.uk/en/products/detail/samsung-electro-mechanics/CL31A106KOHNNNE/3886795?s=N4IgTCBcDaIIxgOwDYC0c4GZHtQOQBEQBdAXyA" (id 8) (at 33.02 53.34 0)
+      (effects (font (size 1.27 1.27)) hide)
+    )
+    (property "Height" "2" (id 9) (at 33.02 53.34 0)
       (effects (font (size 1.27 1.27)) hide)
     )
@@
       (effects (font (size 1.27 1.27)) hide)
     )
-    (property "Mouser #" "" (id 8) (at 153.67 114.3 0)
-      (effects (font (size 1.27 1.27)) hide)
-    )
-    (property "Mouser Part Number" "511-ULN2803A" (id 9) (at 153.67 114.3 0)
+    (property "Mouser #" "511-ULN2803A" (id 8) (at 153.67 114.3 0)
+      (effects (font (size 1.27 1.27)) hide)
+    )
+    (property "Mouser Part Number" "" (id 9) (at 153.67 114.3 0)
+      (effects (font (size 1.27 1.27)) hide)
+    )
+    (property "Height" "5" (id 10) (at 153.67 114.3 0)
       (effects (font (size 1.27 1.27)) hide)
     )
@@
       (effects (font (size 1.27 1.27)) hide)
     )
+    (property "Height" "5" (id 4) (at 113.03 44.45 0)
+      (effects (font (size 1.27 1.27)) hide)
+    )
     (pin "1")
     (pin "10")
@@
       (effects (font (size 1.27 1.27)) hide)
     )
-    (property "Datasheet" "https://www.we-online.com/katalog/datasheet/885012108018.pdf" (id 3) (at 48.26 83.82 0)
-      (effects (font (size 1.27 1.27)) hide)
-    )
-    (property "Manufacturer #" "885012108018" (id 4) (at 48.26 83.82 0)
-      (effects (font (size 1.27 1.27)) hide)
-    )
-    (property "DigiKey #" "732-7642-1-ND" (id 5) (at 48.26 83.82 0)
-      (effects (font (size 1.27 1.27)) hide)
-    )
-    (property "Manufacturer" "Würth Elektronik" (id 6) (at 48.26 83.82 0)
+    (property "Datasheet" "https://media.digikey.com/pdf/Data%20Sheets/Samsung%20PDFs/CL31B106KOHNNNE_Spec.pdf" (id 3) (at 48.26 83.82 0)
+      (effects (font (size 1.27 1.27)) hide)
+    )
+    (property "Manufacturer #" "CL31A226KOHNNNE" (id 4) (at 48.26 83.82 0)
+      (effects (font (size 1.27 1.27)) hide)
+    )
+    (property "DigiKey #" "1276-3048-1-ND" (id 5) (at 48.26 83.82 0)
+      (effects (font (size 1.27 1.27)) hide)
+    )
+    (property "Manufacturer" "Samsung Electro-Mechanics" (id 6) (at 48.26 83.82 0)
       (effects (font (size 1.27 1.27)) hide)
     )
@@
       (effects (font (size 1.27 1.27)) hide)
     )
-    (property "DigiKey Price/Stock" "https://www.digikey.co.uk/en/products/detail/w%C3%BCrth-elektronik/885012108018/5453497?s=N4IgTCBcDaIOwGYwFo4DYAsKCMyByAIiALoC%2BQA" (id 8) (at 48.26 83.82 0)
+    (property "DigiKey Price/Stock" "https://www.digikey.co.uk/en/products/detail/samsung-electro-mechanics/CL31A226KOHNNNE/3888706" (id 8) (at 48.26 83.82 0)
+      (effects (font (size 1.27 1.27)) hide)
+    )
+    (property "Height" "2" (id 9) (at 48.26 83.82 0)
       (effects (font (size 1.27 1.27)) hide)
     )
@@
     )
     (property "Datasheet" "http://www.ti.com/lit/ds/symlink/sn74hc595.pdf" (id 3) (at 113.03 101.6 0)
+      (effects (font (size 1.27 1.27)) hide)
+    )
+    (property "Height" "5" (id 4) (at 113.03 101.6 0)
       (effects (font (size 1.27 1.27)) hide)
     )
@@
       (effects (font (size 1.27 1.27)) hide)
     )
-    (property "Mouser #" "" (id 8) (at 153.67 57.15 0)
-      (effects (font (size 1.27 1.27)) hide)
-    )
-    (property "Mouser Part Number" "511-ULN2803A" (id 9) (at 153.67 57.15 0)
-      (effects (font (size 1.27 1.27)) hide)
-    )
+    (property "Mouser #" "511-ULN2803A" (id 8) (at 153.67 57.15 0)
+      (effects (font (size 1.27 1.27)) hide)
+    )
+    (property "Mouser Part Number" "" (id 9) (at 153.67 57.15 0)
+      (effects (font (size 1.27 1.27)) hide)
+    )
+    (property "Height" "5" (id 10) (at 153.67 57.15 0)
+      (effects (font (size 1.27 1.27)) hide)
+    )
