File: CIB_Main_PCB - Mimic Octopus/Cross Point Matix Ch5-16.kicad_sch (KiCad schematic)
At the start: 7 parts, among them U11 MCP23017_SO, U13 ULN2803A, U15 ULN2803A

Commit message: added changes
Parts:
- removed U11: MCP23017_SO, Package_SO:SOIC-28W_7.5x17.9mm_P1.27mm, symbol Interface_Expansion:MCP23017_SO
- removed U15: ULN2803A, Package_DIP:DIP-18_W7.62mm_LongPads, symbol Transistor_Array:ULN2803A
- added U14, U16: 74HC595, Package_DIP:DIP-16_W7.62mm_LongPads, symbol 74xx:74HC595
- added U23: ULN2803A, Package_DIP:DIP-18_W7.62mm_LongPads, symbol Transistor_Array:ULN2803A
- renumbered C32 to C36, C33 to C37, C34 to C38, C35 to C39
Connections:
- net +12V: now also U23.10 (COM)
- net +5V: now also U14.10 (~{SRCLR}), U14.16 (VCC), U16.10 (~{SRCLR}), U16.16 (VCC)
- net Cross Point Matrix 8 Relays (Med Current) b/Relay 1: now also U23.18 (O1)
- net Cross Point Matrix 8 Relays (Med Current) b/Relay 2: now also U23.17 (O2)
- net Cross Point Matrix 8 Relays (Med Current) b/Relay 3: now also U23.16 (O3)
- net Cross Point Matrix 8 Relays (Med Current) b/Relay 4: now also U23.15 (O4)
- net Cross Point Matrix 8 Relays (Med Current) b/Relay 5: now also U23.14 (O5)
- net Cross Point Matrix 8 Relays (Med Current) b/Relay 6: now also U23.13 (O6)
- net Cross Point Matrix 8 Relays (Med Current) b/Relay 7: now also U23.12 (O7)
- net Cross Point Matrix 8 Relays (Med Current) b/Relay 8: now also U23.11 (O8)
- net GND: now also U14.13 (~{OE}), U14.8 (GND), U16.13 (~{OE}), U16.8 (GND), U23.9 (GND)
- net at U13.8 (I8): now also U14.15 (QA)
- net at U13.7 (I7): now also U14.1 (QB)
- net at U13.6 (I6): now also U14.2 (QC)
- net at U13.5 (I5): now also U14.3 (QD)
- net at U13.4 (I4): now also U14.4 (QE)
- net at U13.3 (I3): now also U14.5 (QF)
- net at U13.2 (I2): now also U14.6 (QG)
- net at U13.1 (I1): now also U14.7 (QH)
- new net: U16.7 (QH), U23.1 (I1)
- new net: U16.6 (QG), U23.2 (I2)
- new net: U16.5 (QF), U23.3 (I3)
- new net: U16.4 (QE), U23.4 (I4)
- new net: U16.3 (QD), U23.5 (I5)
- new net: U16.2 (QC), U23.6 (I6)
- new net: U16.1 (QB), U23.7 (I7)
- new net: U16.15 (QA), U23.8 (I8)
- new net: U14.9 (QH'), U16.14 (SER)
- new net Clock: U14.11 (SRCLK), U16.11 (SRCLK)
- new net DIN: U14.14 (SER)
- new net DOUT: U16.9 (QH')
- new net Latch: U14.12 (RCLK), U16.12 (RCLK)
Other:
- moved on the sheet: U13

Commit message: BoM
Parts:
- C36, C38: Height (none) -> 2
- C37, C39: DigiKey # 732-7642-1-ND -> 1276-3048-1-ND; DigiKey Price/Stock https://www.digikey.co.uk/en/products/detail/w%C3%BCrth-ele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 -> https://www.digikey.co.uk/en/products/detail/samsung-electr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; Height (none) -> 2; Manufacturer Würth Elektronik -> Samsung Electro-Mechanics; Manufacturer # 885012108018 -> CL31A226KOHNNNE
- U13, U23: Height (none) -> 5; Mouser # (none) -> 511-ULN2803A; Mouser Part Number 511-ULN2803A -> (none)
- U14, U16: Height (none) -> 5
Changed lines of the file:
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@@
+      (effects (font (size 1.27 1.27)) hide)
+    )
+    (property "Height" "2" (id 9) (at 33.02 53.34 0)
       (effects (font (size 1.27 1.27)) hide)
     )
@@
       (effects (font (size 1.27 1.27)) hide)
     )
-    (property "Datasheet" "https://www.we-online.com/katalog/datasheet/885012108018.pdf" (id 3) (at 48.26 83.82 0)
-      (effects (font (size 1.27 1.27)) hide)
-    )
-    (property "Manufacturer #" "885012108018" (id 4) (at 48.26 83.82 0)
-      (effects (font (size 1.27 1.27)) hide)
-    )
-    (property "DigiKey #" "732-7642-1-ND" (id 5) (at 48.26 83.82 0)
-      (effects (font (size 1.27 1.27)) hide)
-    )
-    (property "Manufacturer" "Würth Elektronik" (id 6) (at 48.26 83.82 0)
+    (property "Datasheet" "https://media.digikey.com/pdf/Data%20Sheets/Samsung%20PDFs/CL31B106KOHNNNE_Spec.pdf" (id 3) (at 48.26 83.82 0)
+      (effects (font (size 1.27 1.27)) hide)
+    )
+    (property "Manufacturer #" "CL31A226KOHNNNE" (id 4) (at 48.26 83.82 0)
+      (effects (font (size 1.27 1.27)) hide)
+    )
+    (property "DigiKey #" "1276-3048-1-ND" (id 5) (at 48.26 83.82 0)
+      (effects (font (size 1.27 1.27)) hide)
+    )
+    (property "Manufacturer" "Samsung Electro-Mechanics" (id 6) (at 48.26 83.82 0)
       (effects (font (size 1.27 1.27)) hide)
     )
@@
       (effects (font (size 1.27 1.27)) hide)
     )
-    (property "DigiKey Price/Stock" "https://www.digikey.co.uk/en/products/detail/w%C3%BCrth-elektronik/885012108018/5453497?s=N4IgTCBcDaIOwGYwFo4DYAsKCMyByAIiALoC%2BQA" (id 8) (at 48.26 83.82 0)
+    (property "DigiKey Price/Stock" "https://www.digikey.co.uk/en/products/detail/samsung-electro-mechanics/CL31A226KOHNNNE/3888706" (id 8) (at 48.26 83.82 0)
+      (effects (font (size 1.27 1.27)) hide)
+    )
+    (property "Height" "2" (id 9) (at 48.26 83.82 0)
       (effects (font (size 1.27 1.27)) hide)
     )
@@
     )
     (property "DigiKey Price/Stock" "https://www.digikey.co.uk/en/products/detail/samsung-electro-mechanics/CL31A106KOHNNNE/3886795?s=N4IgTCBcDaIIxgOwDYC0c4GZHtQOQBEQBdAXyA" (id 8) (at 33.02 83.82 0)
+      (effects (font (size 1.27 1.27)) hide)
+    )
+    (property "Height" "2" (id 9) (at 33.02 83.82 0)
       (effects (font (size 1.27 1.27)) hide)
     )
@@
       (effects (font (size 1.27 1.27)) hide)
     )
-    (property "Mouser #" "" (id 8) (at 146.05 115.57 0)
-      (effects (font (size 1.27 1.27)) hide)
-    )
-    (property "Mouser Part Number" "511-ULN2803A" (id 9) (at 146.05 115.57 0)
+    (property "Mouser #" "511-ULN2803A" (id 8) (at 146.05 115.57 0)
+      (effects (font (size 1.27 1.27)) hide)
+    )
+    (property "Mouser Part Number" "" (id 9) (at 146.05 115.57 0)
+      (effects (font (size 1.27 1.27)) hide)
+    )
+    (property "Height" "5" (id 10) (at 146.05 115.57 0)
       (effects (font (size 1.27 1.27)) hide)
     )
@@
       (effects (font (size 1.27 1.27)) hide)
     )
-    (property "Mouser #" "" (id 8) (at 146.05 58.42 0)
-      (effects (font (size 1.27 1.27)) hide)
-    )
-    (property "Mouser Part Number" "511-ULN2803A" (id 9) (at 146.05 58.42 0)
+    (property "Mouser #" "511-ULN2803A" (id 8) (at 146.05 58.42 0)
+      (effects (font (size 1.27 1.27)) hide)
+    )
+    (property "Mouser Part Number" "" (id 9) (at 146.05 58.42 0)
+      (effects (font (size 1.27 1.27)) hide)
+    )
+    (property "Height" "5" (id 10) (at 146.05 58.42 0)
       (effects (font (size 1.27 1.27)) hide)
     )
@@
       (effects (font (size 1.27 1.27)) hide)
     )
+    (property "Height" "5" (id 4) (at 105.41 45.72 0)
+      (effects (font (size 1.27 1.27)) hide)
+    )
     (pin "1")
     (pin "10")
@@
       (effects (font (size 1.27 1.27)) hide)
     )
+    (property "Height" "5" (id 4) (at 105.41 102.87 0)
+      (effects (font (size 1.27 1.27)) hide)
+    )
     (pin "1")
     (pin "10")
@@
       (effects (font (size 1.27 1.27)) hide)
     )
-    (property "Datasheet" "https://www.we-online.com/katalog/datasheet/885012108018.pdf" (id 3) (at 48.26 53.34 0)
-      (effects (font (size 1.27 1.27)) hide)
-    )
-    (property "Manufacturer #" "885012108018" (id 4) (at 48.26 53.34 0)
-      (effects (font (size 1.27 1.27)) hide)
-    )
-    (property "DigiKey #" "732-7642-1-ND" (id 5) (at 48.26 53.34 0)
-      (effects (font (size 1.27 1.27)) hide)
-    )
-    (property "Manufacturer" "Würth Elektronik" (id 6) (at 48.26 53.34 0)
+    (property "Datasheet" "https://media.digikey.com/pdf/Data%20Sheets/Samsung%20PDFs/CL31B106KOHNNNE_Spec.pdf" (id 3) (at 48.26 53.34 0)
+      (effects (font (size 1.27 1.27)) hide)
+    )
+    (property "Manufacturer #" "CL31A226KOHNNNE" (id 4) (at 48.26 53.34 0)
+      (effects (font (size 1.27 1.27)) hide)
+    )
+    (property "DigiKey #" "1276-3048-1-ND" (id 5) (at 48.26 53.34 0)
+      (effects (font (size 1.27 1.27)) hide)
+    )
+    (property "Manufacturer" "Samsung Electro-Mechanics" (id 6) (at 48.26 53.34 0)
       (effects (font (size 1.27 1.27)) hide)
     )
@@
       (effects (font (size 1.27 1.27)) hide)
     )
-    (property "DigiKey Price/Stock" "https://www.digikey.co.uk/en/products/detail/w%C3%BCrth-elektronik/885012108018/5453497?s=N4IgTCBcDaIOwGYwFo4DYAsKCMyByAIiALoC%2BQA" (id 8) (at 48.26 53.34 0)
-      (effects (font (size 1.27 1.27)) hide)
-    )
+    (property "DigiKey Price/Stock" "https://www.digikey.co.uk/en/products/detail/samsung-electro-mechanics/CL31A226KOHNNNE/3888706" (id 8) (at 48.26 53.34 0)
+      (effects (font (size 1.27 1.27)) hide)
+    )
+    (property "Height" "2" (id 9) (at 48.26 53.34 0)
+      (effects (font (size 1.27 1.27)) hide)
+    )
