File: CIB_Main_PCB - Mimic Octopus/Cross Point Matrix 8 Relays (High Current).kicad_sch (KiCad schematic)
At the start: 24 parts, among them K64 PC357, K65 PC357, K66 PC357, K67 PC357, K68 PC357, K69 PC357, K70 PC357, K71 PC357

Commit message: added changes
Parts:
- K52: renamed from K64; footprint Connectors:PC375 -> _Connectors:PC375
- K53: renamed from K65; footprint Connectors:PC375 -> _Connectors:PC375
- K54: renamed from K66; footprint Connectors:PC375 -> _Connectors:PC375
- K55: renamed from K67; footprint Connectors:PC375 -> _Connectors:PC375
- K56: renamed from K68; footprint Connectors:PC375 -> _Connectors:PC375
- K57: renamed from K69; footprint Connectors:PC375 -> _Connectors:PC375
- K58: renamed from K70; footprint Connectors:PC375 -> _Connectors:PC375
- K59: renamed from K71; footprint Connectors:PC375 -> _Connectors:PC375
- renumbered D82 to D64, D83 to D65, D84 to D66, D85 to D67, D86 to D68, D87 to D69, D88 to D70, D89 to D71, R147 to R107, R148 to R108, R149 to R109, R150 to R110, R151 to R111, R152 to R112, R153 to R113, R154 to R114

Commit message: BoM
Parts:
- D64, D65, D66, D67, D68, D69, D70, D71: DigiKey Price/Stock (none) -> https://www.digikey.co.uk/en/products/detail/w%C3%BCrth-ele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; Height (none) -> 2
- K52, K53, K54, K55, K56, K57, K58, K59: DigiKey Price/Stock (none) -> https://www.digikey.co.uk/en/products/detail/picker-compone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
Changed lines of the file:
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@@
+      (effects (font (size 1.27 1.27)) hide)
+    )
+    (property "Description" "General Purpose Relay DPDT (2 Form C) 12VDC Coil Through Hole" (id 10) (at 173.99 124.46 0)
+      (effects (font (size 1.27 1.27)) hide)
+    )
+    (property "DigiKey Price/Stock" "https://www.digikey.co.uk/en/products/detail/picker-components/PC375-2C-12S4-X/12352856?s=N4IgTCBcDa4GwGYAsBaACgYQQdgKwrAxQEYwBlVADRQDkAREAXQF8g" (id 11) (at 173.99 124.46 0)
       (effects (font (size 1.27 1.27)) hide)
     )
@@
       (effects (font (size 1.27 1.27)) hide)
     )
+    (property "DigiKey Price/Stock" "https://www.digikey.co.uk/en/products/detail/w%C3%BCrth-elektronik/150120VS75000/4489945?s=N4IgTCBcDaIOwGYwFoAsBOdDkEZkDkAREAXQF8g" (id 13) (at 127 143.51 0)
+      (effects (font (size 1.27 1.27)) hide)
+    )
+    (property "Height" "2" (id 14) (at 127 143.51 0)
+      (effects (font (size 1.27 1.27)) hide)
+    )
     (pin "1")
     (pin "2")
@@
       (effects (font (size 1.27 1.27)) hide)
     )
+    (property "DigiKey Price/Stock" "https://www.digikey.co.uk/en/products/detail/w%C3%BCrth-elektronik/150120VS75000/4489945?s=N4IgTCBcDaIOwGYwFoAsBOdDkEZkDkAREAXQF8g" (id 13) (at 228.6 92.71 0)
+      (effects (font (size 1.27 1.27)) hide)
+    )
+    (property "Height" "2" (id 14) (at 228.6 92.71 0)
+      (effects (font (size 1.27 1.27)) hide)
+    )
     (pin "1")
     (pin "2")
@@
       (effects (font (size 1.27 1.27)) hide)
     )
+    (property "DigiKey Price/Stock" "https://www.digikey.co.uk/en/products/detail/w%C3%BCrth-elektronik/150120VS75000/4489945?s=N4IgTCBcDaIOwGYwFoAsBOdDkEZkDkAREAXQF8g" (id 13) (at 76.2 92.71 0)
+      (effects (font (size 1.27 1.27)) hide)
+    )
+    (property "Height" "2" (id 14) (at 76.2 92.71 0)
+      (effects (font (size 1.27 1.27)) hide)
+    )
     (pin "1")
     (pin "2")
@@
     )
     (property "Manufacturer" "Picker Components" (id 9) (at 224.79 73.66 0)
+      (effects (font (size 1.27 1.27)) hide)
+    )
+    (property "Description" "General Purpose Relay DPDT (2 Form C) 12VDC Coil Through Hole" (id 10) (at 224.79 73.66 0)
+      (effects (font (size 1.27 1.27)) hide)
+    )
+    (property "DigiKey Price/Stock" "https://www.digikey.co.uk/en/products/detail/picker-components/PC375-2C-12S4-X/12352856?s=N4IgTCBcDa4GwGYAsBaACgYQQdgKwrAxQEYwBlVADRQDkAREAXQF8g" (id 11) (at 224.79 73.66 0)
       (effects (font (size 1.27 1.27)) hide)
     )
@@
       (effects (font (size 1.27 1.27)) hide)
     )
+    (property "Description" "General Purpose Relay DPDT (2 Form C) 12VDC Coil Through Hole" (id 10) (at 72.39 124.46 0)
+      (effects (font (size 1.27 1.27)) hide)
+    )
+    (property "DigiKey Price/Stock" "https://www.digikey.co.uk/en/products/detail/picker-components/PC375-2C-12S4-X/12352856?s=N4IgTCBcDa4GwGYAsBaACgYQQdgKwrAxQEYwBlVADRQDkAREAXQF8g" (id 11) (at 72.39 124.46 0)
+      (effects (font (size 1.27 1.27)) hide)
+    )
     (pin "1")
     (pin "2")
@@
       (effects (font (size 1.27 1.27)) hide)
     )
+    (property "Description" "General Purpose Relay DPDT (2 Form C) 12VDC Coil Through Hole" (id 10) (at 224.79 124.46 0)
+      (effects (font (size 1.27 1.27)) hide)
+    )
+    (property "DigiKey Price/Stock" "https://www.digikey.co.uk/en/products/detail/picker-components/PC375-2C-12S4-X/12352856?s=N4IgTCBcDa4GwGYAsBaACgYQQdgKwrAxQEYwBlVADRQDkAREAXQF8g" (id 11) (at 224.79 124.46 0)
+      (effects (font (size 1.27 1.27)) hide)
+    )
     (pin "1")
     (pin "2")
@@
       (effects (font (size 1.27 1.27)) hide)
     )
+    (property "DigiKey Price/Stock" "https://www.digikey.co.uk/en/products/detail/w%C3%BCrth-elektronik/150120VS75000/4489945?s=N4IgTCBcDaIOwGYwFoAsBOdDkEZkDkAREAXQF8g" (id 13) (at 127 92.71 0)
+      (effects (font (size 1.27 1.27)) hide)
+    )
+    (property "Height" "2" (id 14) (at 127 92.71 0)
+      (effects (font (size 1.27 1.27)) hide)
+    )
     (pin "1")
     (pin "2")
@@
       (effects (font (size 1.27 1.27)) hide)
     )
+    (property "DigiKey Price/Stock" "https://www.digikey.co.uk/en/products/detail/w%C3%BCrth-elektronik/150120VS75000/4489945?s=N4IgTCBcDaIOwGYwFoAsBOdDkEZkDkAREAXQF8g" (id 13) (at 228.6 143.51 0)
+      (effects (font (size 1.27 1.27)) hide)
+    )
+    (property "Height" "2" (id 14) (at 228.6 143.51 0)
+      (effects (font (size 1.27 1.27)) hide)
+    )
     (pin "1")
     (pin "2")
@@
     )
     (property "Manufacturer" "Picker Components" (id 9) (at 72.39 73.66 0)
+      (effects (font (size 1.27 1.27)) hide)
+    )
+    (property "Description" "General Purpose Relay DPDT (2 Form C) 12VDC Coil Through Hole" (id 10) (at 72.39 73.66 0)
+      (effects (font (size 1.27 1.27)) hide)
+    )
+    (property "DigiKey Price/Stock" "https://www.digikey.co.uk/en/products/detail/picker-components/PC375-2C-12S4-X/12352856?s=N4IgTCBcDa4GwGYAsBaACgYQQdgKwrAxQEYwBlVADRQDkAREAXQF8g" (id 11) (at 72.39 73.66 0)
       (effects (font (size 1.27 1.27)) hide)
     )
@@
       (effects (font (size 1.27 1.27)) hide)
     )
+    (property "DigiKey Price/Stock" "https://www.digikey.co.uk/en/products/detail/w%C3%BCrth-elektronik/150120VS75000/4489945?s=N4IgTCBcDaIOwGYwFoAsBOdDkEZkDkAREAXQF8g" (id 13) (at 76.2 143.51 0)
+      (effects (font (size 1.27 1.27)) hide)
+    )
+    (property "Height" "2" (id 14) (at 76.2 143.51 0)
+      (effects (font (size 1.27 1.27)) hide)
+    )
     (pin "1")
     (pin "2")
@@
       (effects (font (size 1.27 1.27)) hide)
     )
+    (property "DigiKey Price/Stock" "https://www.digikey.co.uk/en/products/detail/w%C3%BCrth-elektronik/150120VS75000/4489945?s=N4IgTCBcDaIOwGYwFoAsBOdDkEZkDkAREAXQF8g" (id 13) (at 177.8 143.51 0)
+      (effects (font (size 1.27 1.27)) hide)
+    )
+    (property "Height" "2" (id 14) (at 177.8 143.51 0)
+      (effects (font (size 1.27 1.27)) hide)
+    )
     (pin "1")
     (pin "2")
@@
       (effects (font (size 1.27 1.27)) hide)
     )
+    (property "DigiKey Price/Stock" "https://www.digikey.co.uk/en/products/detail/w%C3%BCrth-elektronik/150120VS75000/4489945?s=N4IgTCBcDaIOwGYwFoAsBOdDkEZkDkAREAXQF8g" (id 13) (at 177.8 92.71 0)
+      (effects (font (size 1.27 1.27)) hide)
+    )
+    (property "Height" "2" (id 14) (at 177.8 92.71 0)
+      (effects (font (size 1.27 1.27)) hide)
+    )
     (pin "1")
     (pin "2")
@@
     )
     (property "Manufacturer" "Picker Components" (id 9) (at 173.99 73.66 0)
+      (effects (font (size 1.27 1.27)) hide)
+    )
+    (property "Description" "General Purpose Relay DPDT (2 Form C) 12VDC Coil Through Hole" (id 10) (at 173.99 73.66 0)
+      (effects (font (size 1.27 1.27)) hide)
+    )
+    (property "DigiKey Price/Stock" "https://www.digikey.co.uk/en/products/detail/picker-components/PC375-2C-12S4-X/12352856?s=N4IgTCBcDa4GwGYAsBaACgYQQdgKwrAxQEYwBlVADRQDkAREAXQF8g" (id 11) (at 173.99 73.66 0)
       (effects (font (size 1.27 1.27)) hide)
     )
@@
       (effects (font (size 1.27 1.27)) hide)
     )
+    (property "Description" "General Purpose Relay DPDT (2 Form C) 12VDC Coil Through Hole" (id 10) (at 123.19 124.46 0)
+      (effects (font (size 1.27 1.27)) hide)
+    )
+    (property "DigiKey Price/Stock" "https://www.digikey.co.uk/en/products/detail/picker-components/PC375-2C-12S4-X/12352856?s=N4IgTCBcDa4GwGYAsBaACgYQQdgKwrAxQEYwBlVADRQDkAREAXQF8g" (id 11) (at 123.19 124.46 0)
+      (effects (font (size 1.27 1.27)) hide)
+    )
     (pin "1")
     (pin "2")
@@
       (effects (font (size 1.27 1.27)) hide)
     )
+    (property "Description" "General Purpose Relay DPDT (2 Form C) 12VDC Coil Through Hole" (id 10) (at 123.19 73.66 0)
+      (effects (font (size 1.27 1.27)) hide)
+    )
+    (property "DigiKey Price/Stock" "https://www.digikey.co.uk/en/products/detail/picker-components/PC375-2C-12S4-X/12352856?s=N4IgTCBcDa4GwGYAsBaACgYQQdgKwrAxQEYwBlVADRQDkAREAXQF8g" (id 11) (at 123.19 73.66 0)
+      (effects (font (size 1.27 1.27)) hide)
+    )

Commit message: changes
Parts:
- removed D64, D65, D66, D67, D68, D69, D70, D71: Green, Diode_SMD:D_1206_3216Metric_Pad1.42x1.75mm_HandSolder, symbol Device:LED_Small_Filled
- removed R107, R108, R109, R110, R111, R112, R113, R114: 1k2, Resistor_SMD:R_1206_3216Metric_Pad1.30x1.75mm_HandSolder, symbol Device:R_Small
