File: CIB_Main_PCB - Mimic Octopus/Cross Point Matrix 8 Relays (Low Current).kicad_sch (KiCad schematic)
At the start: 24 parts

Commit message: added changes
Parts:
- renumbered D69 to D47, D70 to D48, D71 to D49, D72 to D50, D73 to D51, D74 to D52, D75 to D53, D76 to D54, K54 to K42, K55 to K43, K56 to K44, K57 to K45, K58 to K46, K59 to K47, K60 to K48, K61 to K49, R129 to R74, R130 to R75, R131 to R76, R132 to R77, R133 to R78, R134 to R79, R135 to R80, R136 to R81

Commit message: BoM
Parts:
- D47, D48, D49, D50, D51, D52, D53, D54: DigiKey Price/Stock (none) -> https://www.digikey.co.uk/en/products/detail/w%C3%BCrth-ele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; Height (none) -> 2
- K42, K43, K44, K45, K46, K47, K48, K49: value ~ -> G6K-2P DC12; DigiKey Price/Stock (none) -> https://www.digikey.co.uk/en/products/detail/omron-electron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; Manufacture Omron Electronics Inc-EMC Div -> (none); Manufacturer (none) -> Omron Electronics Inc-EMC Div

Commit message: changes
Parts:
- removed D47, D48, D49, D50, D51, D52, D53, D54: Green, Diode_SMD:D_1206_3216Metric_Pad1.42x1.75mm_HandSolder, symbol Device:LED_Small_Filled
- removed R74, R75, R76, R77, R78, R79, R80, R81: 1k2, Resistor_SMD:R_1206_3216Metric_Pad1.30x1.75mm_HandSolder, symbol Device:R_Small
- K42, K43, K44, K45, K46, K47, K48, K49: value G6K-2P DC12 -> PC357; footprint Relay_THT:Relay_DPDT_Omron_G6K-2P -> _Connectors:PC375; DigiKey # Z117-ND -> 2634-PC375-2C-12S4-X-ND; DigiKey Price/Stock https://www.digikey.co.uk/en/products/detail/omron-electron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 -> https://www.digikey.co.uk/en/products/detail/picker-compone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; Manufacturer Omron Electronics Inc-EMC Div -> Picker Components; Manufacturer # G6K-2P DC12 -> PC375-2C-12S4-X
