File: CIB_Main_PCB - Mimic Octopus/Cross Point Matrix 8 Relays (Med Current).kicad_sch (KiCad schematic)
At the start: 24 parts, among them K72 G2RL, K73 G2RL, K74 G2RL, K75 G2RL, K76 G2RL, K77 G2RL, K78 G2RL, K79 G2RL

Commit message: added changes
Parts:
- renumbered D90 to D80, D91 to D81, D92 to D82, D93 to D83, D94 to D84, D95 to D85, D96 to D86, D97 to D87, K72 to K68, K73 to K69, K74 to K70, K75 to K71, K76 to K72, K77 to K73, K78 to K74, K79 to K75, R155 to R123, R156 to R124, R157 to R125, R158 to R126, R159 to R127, R160 to R128, R161 to R129, R162 to R130

Commit message: BoM
Parts:
- D80, D81, D82, D83, D84, D85, D86, D87: DigiKey Price/Stock (none) -> https://www.digikey.co.uk/en/products/detail/w%C3%BCrth-ele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; Height (none) -> 2
- K68, K69, K70, K71, K72, K73, K74, K75: value G2RL -> G6K-2P DC12
Changed lines of the file:
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@@
+      (effects (font (size 1.27 1.27)) hide)
+    )
+    (property "DigiKey Price/Stock" "https://www.digikey.co.uk/en/products/detail/w%C3%BCrth-elektronik/150120VS75000/4489945?s=N4IgTCBcDaIOwGYwFoAsBOdDkEZkDkAREAXQF8g" (id 13) (at 177.8 92.71 0)
+      (effects (font (size 1.27 1.27)) hide)
+    )
+    (property "Height" "2" (id 14) (at 177.8 92.71 0)
       (effects (font (size 1.27 1.27)) hide)
     )
@@
     (in_bom yes) (on_board yes) (fields_autoplaced)
     (property "Reference" "K71" (id 0) (at 224.79 52.832 90))
-    (property "Value" "G2RL" (id 1) (at 224.79 55.372 90)
+    (property "Value" "G6K-2P DC12" (id 1) (at 224.79 55.372 90)
       (effects (font (size 1.27 1.27)) hide)
     )
@@
     )
     (property "Manufacturer" "Omron Electronics Inc-EMC Div" (id 9) (at 224.79 73.66 0)
+      (effects (font (size 1.27 1.27)) hide)
+    )
+    (property "Description" "Telecom Relay DPDT (2 Form C) Through Hole" (id 10) (at 224.79 73.66 0)
       (effects (font (size 1.27 1.27)) hide)
     )
@@
       (effects (font (size 1.27 1.27)) hide)
     )
+    (property "DigiKey Price/Stock" "https://www.digikey.co.uk/en/products/detail/w%C3%BCrth-elektronik/150120VS75000/4489945?s=N4IgTCBcDaIOwGYwFoAsBOdDkEZkDkAREAXQF8g" (id 13) (at 76.2 92.71 0)
+      (effects (font (size 1.27 1.27)) hide)
+    )
+    (property "Height" "2" (id 14) (at 76.2 92.71 0)
+      (effects (font (size 1.27 1.27)) hide)
+    )
     (pin "1")
     (pin "2")
@@
     (in_bom yes) (on_board yes) (fields_autoplaced)
     (property "Reference" "K69" (id 0) (at 123.19 52.832 90))
-    (property "Value" "G2RL" (id 1) (at 123.19 55.372 90)
+    (property "Value" "G6K-2P DC12" (id 1) (at 123.19 55.372 90)
       (effects (font (size 1.27 1.27)) hide)
     )
@@
     )
     (property "Manufacturer" "Omron Electronics Inc-EMC Div" (id 9) (at 123.19 73.66 0)
+      (effects (font (size 1.27 1.27)) hide)
+    )
+    (property "Description" "Telecom Relay DPDT (2 Form C) Through Hole" (id 10) (at 123.19 73.66 0)
       (effects (font (size 1.27 1.27)) hide)
     )
@@
       (effects (font (size 1.27 1.27)) hide)
     )
+    (property "DigiKey Price/Stock" "https://www.digikey.co.uk/en/products/detail/w%C3%BCrth-elektronik/150120VS75000/4489945?s=N4IgTCBcDaIOwGYwFoAsBOdDkEZkDkAREAXQF8g" (id 13) (at 76.2 143.51 0)
+      (effects (font (size 1.27 1.27)) hide)
+    )
+    (property "Height" "2" (id 14) (at 76.2 143.51 0)
+      (effects (font (size 1.27 1.27)) hide)
+    )
     (pin "1")
     (pin "2")
@@
       (effects (font (size 1.27 1.27)) hide)
     )
+    (property "DigiKey Price/Stock" "https://www.digikey.co.uk/en/products/detail/w%C3%BCrth-elektronik/150120VS75000/4489945?s=N4IgTCBcDaIOwGYwFoAsBOdDkEZkDkAREAXQF8g" (id 13) (at 228.6 143.51 0)
+      (effects (font (size 1.27 1.27)) hide)
+    )
+    (property "Height" "2" (id 14) (at 228.6 143.51 0)
+      (effects (font (size 1.27 1.27)) hide)
+    )
     (pin "1")
     (pin "2")
@@
       (effects (font (size 1.27 1.27)) hide)
     )
+    (property "DigiKey Price/Stock" "https://www.digikey.co.uk/en/products/detail/w%C3%BCrth-elektronik/150120VS75000/4489945?s=N4IgTCBcDaIOwGYwFoAsBOdDkEZkDkAREAXQF8g" (id 13) (at 127 143.51 0)
+      (effects (font (size 1.27 1.27)) hide)
+    )
+    (property "Height" "2" (id 14) (at 127 143.51 0)
+      (effects (font (size 1.27 1.27)) hide)
+    )
     (pin "1")
     (pin "2")
@@
     (in_bom yes) (on_board yes) (fields_autoplaced)
     (property "Reference" "K73" (id 0) (at 123.19 103.632 90))
-    (property "Value" "G2RL" (id 1) (at 123.19 106.172 90)
+    (property "Value" "G6K-2P DC12" (id 1) (at 123.19 106.172 90)
       (effects (font (size 1.27 1.27)) hide)
     )
@@
     )
     (property "Manufacturer" "Omron Electronics Inc-EMC Div" (id 9) (at 123.19 124.46 0)
+      (effects (font (size 1.27 1.27)) hide)
+    )
+    (property "Description" "Telecom Relay DPDT (2 Form C) Through Hole" (id 10) (at 123.19 124.46 0)
       (effects (font (size 1.27 1.27)) hide)
     )
@@
     (in_bom yes) (on_board yes) (fields_autoplaced)
     (property "Reference" "K68" (id 0) (at 72.39 55.88 90))
-    (property "Value" "G2RL" (id 1) (at 72.39 55.372 90)
+    (property "Value" "G6K-2P DC12" (id 1) (at 72.39 55.372 90)
       (effects (font (size 1.27 1.27)) hide)
     )
@@
     )
     (property "Manufacturer" "Omron Electronics Inc-EMC Div" (id 9) (at 72.39 73.66 0)
+      (effects (font (size 1.27 1.27)) hide)
+    )
+    (property "Description" "Telecom Relay DPDT (2 Form C) Through Hole" (id 10) (at 72.39 73.66 0)
       (effects (font (size 1.27 1.27)) hide)
     )
@@
       (effects (font (size 1.27 1.27)) hide)
     )
+    (property "DigiKey Price/Stock" "https://www.digikey.co.uk/en/products/detail/w%C3%BCrth-elektronik/150120VS75000/4489945?s=N4IgTCBcDaIOwGYwFoAsBOdDkEZkDkAREAXQF8g" (id 13) (at 228.6 92.71 0)
+      (effects (font (size 1.27 1.27)) hide)
+    )
+    (property "Height" "2" (id 14) (at 228.6 92.71 0)
+      (effects (font (size 1.27 1.27)) hide)
+    )
     (pin "1")
     (pin "2")
@@
     (in_bom yes) (on_board yes) (fields_autoplaced)
     (property "Reference" "K70" (id 0) (at 173.99 52.832 90))
-    (property "Value" "G2RL" (id 1) (at 173.99 55.372 90)
+    (property "Value" "G6K-2P DC12" (id 1) (at 173.99 55.372 90)
       (effects (font (size 1.27 1.27)) hide)
     )
@@
     )
     (property "Manufacturer" "Omron Electronics Inc-EMC Div" (id 9) (at 173.99 73.66 0)
+      (effects (font (size 1.27 1.27)) hide)
+    )
+    (property "Description" "Telecom Relay DPDT (2 Form C) Through Hole" (id 10) (at 173.99 73.66 0)
       (effects (font (size 1.27 1.27)) hide)
     )
@@
       (effects (font (size 1.27 1.27)) hide)
     )
+    (property "DigiKey Price/Stock" "https://www.digikey.co.uk/en/products/detail/w%C3%BCrth-elektronik/150120VS75000/4489945?s=N4IgTCBcDaIOwGYwFoAsBOdDkEZkDkAREAXQF8g" (id 13) (at 127 92.71 0)
+      (effects (font (size 1.27 1.27)) hide)
+    )
+    (property "Height" "2" (id 14) (at 127 92.71 0)
+      (effects (font (size 1.27 1.27)) hide)
+    )
     (pin "1")
     (pin "2")
@@
     (in_bom yes) (on_board yes) (fields_autoplaced)
     (property "Reference" "K75" (id 0) (at 224.79 103.632 90))
-    (property "Value" "G2RL" (id 1) (at 224.79 106.172 90)
+    (property "Value" "G6K-2P DC12" (id 1) (at 224.79 106.172 90)
       (effects (font (size 1.27 1.27)) hide)
     )
@@
     )
     (property "Manufacturer" "Omron Electronics Inc-EMC Div" (id 9) (at 224.79 124.46 0)
+      (effects (font (size 1.27 1.27)) hide)
+    )
+    (property "Description" "Telecom Relay DPDT (2 Form C) Through Hole" (id 10) (at 224.79 124.46 0)
       (effects (font (size 1.27 1.27)) hide)
     )
@@
       (effects (font (size 1.27 1.27)) hide)
     )
+    (property "DigiKey Price/Stock" "https://www.digikey.co.uk/en/products/detail/w%C3%BCrth-elektronik/150120VS75000/4489945?s=N4IgTCBcDaIOwGYwFoAsBOdDkEZkDkAREAXQF8g" (id 13) (at 177.8 143.51 0)
+      (effects (font (size 1.27 1.27)) hide)
+    )
+    (property "Height" "2" (id 14) (at 177.8 143.51 0)
+      (effects (font (size 1.27 1.27)) hide)
+    )
     (pin "1")
     (pin "2")
@@
     (in_bom yes) (on_board yes) (fields_autoplaced)
     (property "Reference" "K74" (id 0) (at 173.99 103.632 90))
-    (property "Value" "G2RL" (id 1) (at 173.99 106.172 90)
+    (property "Value" "G6K-2P DC12" (id 1) (at 173.99 106.172 90)
       (effects (font (size 1.27 1.27)) hide)
     )
@@
     )
     (property "Manufacturer" "Omron Electronics Inc-EMC Div" (id 9) (at 173.99 124.46 0)
+      (effects (font (size 1.27 1.27)) hide)
+    )
+    (property "Description" "Telecom Relay DPDT (2 Form C) Through Hole" (id 10) (at 173.99 124.46 0)
       (effects (font (size 1.27 1.27)) hide)
     )
@@
     (in_bom yes) (on_board yes) (fields_autoplaced)
     (property "Reference" "K72" (id 0) (at 72.39 103.632 90))
-    (property "Value" "G2RL" (id 1) (at 72.39 106.172 90)
+    (property "Value" "G6K-2P DC12" (id 1) (at 72.39 106.172 90)
       (effects (font (size 1.27 1.27)) hide)
     )
@@
       (effects (font (size 1.27 1.27)) hide)
     )
+    (property "Description" "Telecom Relay DPDT (2 Form C) Through Hole" (id 10) (at 72.39 124.46 0)
+      (effects (font (size 1.27 1.27)) hide)
+    )

Commit message: changes
Parts:
- removed D80, D81, D82, D83, D84, D85, D86, D87: Green, Diode_SMD:D_1206_3216Metric_Pad1.42x1.75mm_HandSolder, symbol Device:LED_Small_Filled
- removed R123, R124, R125, R126, R127, R128, R129, R130: 1k2, Resistor_SMD:R_1206_3216Metric_Pad1.30x1.75mm_HandSolder, symbol Device:R_Small
- K68: value G6K-2P DC12 -> PC357; footprint Relay_THT:Relay_DPDT_Omron_G2RL -> _Connectors:PC375; DigiKey # Z117-ND -> 2634-PC375-2C-12S4-X-ND; DigiKey Price/Stock (none) -> https://www.digikey.co.uk/en/products/detail/picker-compone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; Manufacturer Omron Electronics Inc-EMC Div -> Picker Components; Manufacturer # G6K-2P DC12 -> PC375-2C-12S4-X
- K69, K70, K71, K72, K73, K74, K75: value G6K-2P DC12 -> PC357; footprint Relay_THT:Relay_DPDT_Omron_G2RL -> _Connectors:PC375; DigiKey # Z4267-ND or Z3088-ND -> 2634-PC375-2C-12S4-X-ND; DigiKey Price/Stock (none) -> https://www.digikey.co.uk/en/products/detail/picker-compone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; Manufacturer Omron Electronics Inc-EMC Div -> Picker Components; Manufacturer # G2RL2ADC12BYOMB or G2RL24CFDC12 -> PC375-2C-12S4-X
