File: CIB_Main_PCB - Mimic Octopus/Cross Point Matrix.kicad_sch (KiCad schematic)
At the start: 12 parts, among them J11 Ch 1-4, J18 Ch 13-16, J19 Ch 21-24, J7 Ch 5-8, J8 Ch 9-12, J9 Ch 17-20

Commit message: added changes
Parts:
- removed 0x20, 0x21, 0x22, 0x23, 0x24, 0x25: 10k, Resistor_SMD:R_Array_Convex_4x1206, symbol Device:R_Pack04
- J10: renamed from J7; footprint Component Search Engine:Pluggable Terminal Blocks SDDC 1,5 4-PV-3,5 -> Component Search Engine:Pluggable Terminal Blocks SDDC 1.5mm pitch 8 Pin; symbol Component Search Engine:Pluggable Terminal Blocks SDDC 1,5/ 4-PV-3,5 -> Component Search Engine:Pluggable Terminal Blocks SDDC 1.5mm pitch 8 Pin; Manufacturer_Name (none) -> Phoenix Contact; Manufacturer_Part_Number (none) -> 1848668
- J11: renamed from J8; footprint Component Search Engine:Pluggable Terminal Blocks SDDC 1,5 4-PV-3,5 -> Component Search Engine:Pluggable Terminal Blocks SDDC 1.5mm pitch 8 Pin; symbol Component Search Engine:Pluggable Terminal Blocks SDDC 1,5/ 4-PV-3,5 -> Component Search Engine:Pluggable Terminal Blocks SDDC 1.5mm pitch 8 Pin; Manufacturer_Name (none) -> Phoenix Contact; Manufacturer_Part_Number (none) -> 1848668
- J12: renamed from J18; footprint Component Search Engine:Pluggable Terminal Blocks SDDC 1,5 4-PV-3,5 -> Component Search Engine:Pluggable Terminal Blocks SDDC 1.5mm pitch 8 Pin; symbol Component Search Engine:Pluggable Terminal Blocks SDDC 1,5/ 4-PV-3,5 -> Component Search Engine:Pluggable Terminal Blocks SDDC 1.5mm pitch 8 Pin; Manufacturer_Name (none) -> Phoenix Contact; Manufacturer_Part_Number (none) -> 1848668
- J13: renamed from J9; footprint Component Search Engine:Pluggable Terminal Blocks SDDC 1,5 4-PV-3,5 -> Component Search Engine:Pluggable Terminal Blocks SDDC 1.5mm pitch 8 Pin; symbol Component Search Engine:Pluggable Terminal Blocks SDDC 1,5/ 4-PV-3,5 -> Component Search Engine:Pluggable Terminal Blocks SDDC 1.5mm pitch 8 Pin; Manufacturer_Name (none) -> Phoenix Contact; Manufacturer_Part_Number (none) -> 1848668
- J14: renamed from J19; footprint Component Search Engine:Pluggable Terminal Blocks SDDC 1,5 4-PV-3,5 -> Component Search Engine:Pluggable Terminal Blocks SDDC 1.5mm pitch 8 Pin; symbol Component Search Engine:Pluggable Terminal Blocks SDDC 1,5/ 4-PV-3,5 -> Component Search Engine:Pluggable Terminal Blocks SDDC 1.5mm pitch 8 Pin; Manufacturer_Name (none) -> Phoenix Contact; Manufacturer_Part_Number (none) -> 1848668
- J9: renamed from J11; footprint Component Search Engine:Pluggable Terminal Blocks SDC 2,5 8-PV-5,0 0-ZB -> Component Search Engine:Pluggable Terminal Blocks SDC 2.5mm pitch 8 Pin; symbol Component Search Engine:Pluggable Terminal Blocks SDC 2,5/ 8-PV-5,0 0-ZB -> Component Search Engine:Pluggable Terminal Blocks SDC 2.5mm pitch 8 Pin; Manufacturer_Name (none) -> Phoenix Contact; Manufacturer_Part_Number (none) -> 1864095
Other:
- sheet Cross Point Matrix 8 Relays Ch1-4 (High Current) ports: added Clock, DIN, DOUT, Latch; removed A0, A1, A2, SCL 5V, SDA 5V, ~{RESET}
- sheet Cross Point Matrix 8 Relays Ch13-16 (Med Current) ports: added Clock, DIN, DOUT, Latch; removed A0, A1, A2, SCL 5V, SDA 5V, ~{RESET}
- sheet Cross Point Matrix 8 Relays Ch17-20 (Low Current) ports: added Clock, DIN, DOUT, Latch; removed A0, A1, A2, SCL 5V, SDA 5V, ~{RESET}
- sheet Cross Point Matrix 8 Relays Ch21-24 (Low Current) ports: added Clock, DIN, DOUT, Latch; removed A0, A1, A2, SCL 5V, SDA 5V, ~{RESET}
- sheet Cross Point Matrix 8 Relays Ch5-8 (Med Current) ports: added Clock, DIN, DOUT, Latch; removed A0, A1, A2, SCL 5V, SDA 5V, ~{RESET}
- sheet Cross Point Matrix 8 Relays Ch9-12 (Med Current) ports: added Clock, DIN, DOUT, Latch; removed A0, A1, A2, SCL 5V, SDA 5V, ~{RESET}
- note removed: "0x20"
- note removed: "0x21"
- note removed: "0x22"
- note removed: "0x23"
- note removed: "0x24"
- note removed: "0x25"

Commit message: V0.1 PCB to be sent out
Parts:
- added NT1, NT2, NT3, NT4, NT5, NT6, NT7, NT8: NetTie_2, NetTie:NetTie-2_SMD_Pad0.5mm, symbol Device:NetTie_2
Connections:
- net Eq Ch1 High: now also NT1.2
- net Eq Ch1 Low: now also NT2.2
- net Eq Ch2 High: now also NT3.2
- net Eq Ch2 Low: now also NT4.2
- net Eq Ch3 High: now also NT5.2
- net Eq Ch3 Low: now also NT6.2
- net Eq Ch4 High: now also NT7.2
- net Eq Ch4 Low: now also NT8.2
- new net Eq Ch1 High (low C): NT1.1
- new net Eq Ch1 Low (low C): NT2.1
- new net Eq Ch2 High (low C): NT3.1
- new net Eq Ch2 Low (low C): NT4.1
- new net Eq Ch3 High (low C): NT5.1
- new net Eq Ch3 Low (low C): NT6.1
- new net Eq Ch4 High (low C): NT7.1
- new net Eq Ch4 Low (low C): NT8.1
Other:
- note added: "Net-ties are used to change net size"

Commit message: BoM
Parts:
- J10, J11, J12, J13, J14: Manufacturer_Name Phoenix Contact -> (none); Manufacturer_Part_Number 1848668 -> (none); Mouser # (none) -> 651-1848668; Mouser Part Number 651-1848668 -> (none)
- J9: Manufacturer_Name Phoenix Contact -> (none); Manufacturer_Part_Number 1864095 -> (none); Mouser # (none) -> 651-1864095; Mouser Part Number 651-1864095 -> (none)
- NT1, NT2, NT3, NT4, NT5, NT6, NT7, NT8: dnp (none) -> dnp
Changed lines of the file:
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@@
+      (effects (font (size 1.27 1.27)) hide)
+    )
+    (property "dnp" "dnp" (id 4) (at 204.47 156.21 0)
       (effects (font (size 1.27 1.27)) hide)
     )
@@
       (effects (font (size 1.27 1.27)) (justify left) hide)
     )
-    (property "Manufacturer_Name" "Phoenix Contact" (id 6) (at 262.89 101.6 0)
-      (effects (font (size 1.27 1.27)) (justify left) hide)
-    )
-    (property "Manufacturer_Part_Number" "1848668" (id 7) (at 262.89 104.14 0)
-      (effects (font (size 1.27 1.27)) (justify left) hide)
-    )
-    (property "Mouser Part Number" "651-1848668" (id 8) (at 262.89 106.68 0)
+    (property "Manufacturer_Name" "" (id 6) (at 262.89 101.6 0)
+      (effects (font (size 1.27 1.27)) (justify left) hide)
+    )
+    (property "Manufacturer_Part_Number" "" (id 7) (at 262.89 104.14 0)
+      (effects (font (size 1.27 1.27)) (justify left) hide)
+    )
+    (property "Mouser Part Number" "" (id 8) (at 262.89 106.68 0)
       (effects (font (size 1.27 1.27)) (justify left) hide)
     )
@@
     )
     (property "Manufacturer #" "1848668" (id 13) (at 241.3 93.98 0)
+      (effects (font (size 1.27 1.27)) hide)
+    )
+    (property "Mouser #" "651-1848668" (id 14) (at 241.3 93.98 0)
       (effects (font (size 1.27 1.27)) hide)
     )
@@
       (effects (font (size 1.27 1.27)) (justify left) hide)
     )
-    (property "Manufacturer_Name" "Phoenix Contact" (id 6) (at 262.89 54.61 0)
-      (effects (font (size 1.27 1.27)) (justify left) hide)
-    )
-    (property "Manufacturer_Part_Number" "1848668" (id 7) (at 262.89 57.15 0)
-      (effects (font (size 1.27 1.27)) (justify left) hide)
-    )
-    (property "Mouser Part Number" "651-1848668" (id 8) (at 262.89 59.69 0)
+    (property "Manufacturer_Name" "" (id 6) (at 262.89 54.61 0)
+      (effects (font (size 1.27 1.27)) (justify left) hide)
+    )
+    (property "Manufacturer_Part_Number" "" (id 7) (at 262.89 57.15 0)
+      (effects (font (size 1.27 1.27)) (justify left) hide)
+    )
+    (property "Mouser Part Number" "" (id 8) (at 262.89 59.69 0)
       (effects (font (size 1.27 1.27)) (justify left) hide)
     )
@@
     )
     (property "Manufacturer #" "1848668" (id 13) (at 241.3 46.99 0)
+      (effects (font (size 1.27 1.27)) hide)
+    )
+    (property "Mouser #" "651-1848668" (id 14) (at 241.3 46.99 0)
       (effects (font (size 1.27 1.27)) hide)
     )
@@
       (effects (font (size 1.27 1.27)) hide)
     )
+    (property "dnp" "dnp" (id 4) (at 204.47 158.75 0)
+      (effects (font (size 1.27 1.27)) hide)
+    )
     (pin "1")
     (pin "2")
@@
       (effects (font (size 1.27 1.27)) hide)
     )
+    (property "dnp" "dnp" (id 4) (at 204.47 143.51 0)
+      (effects (font (size 1.27 1.27)) hide)
+    )
     (pin "1")
     (pin "2")
@@
       (effects (font (size 1.27 1.27)) hide)
     )
+    (property "dnp" "dnp" (id 4) (at 204.47 151.13 0)
+      (effects (font (size 1.27 1.27)) hide)
+    )
     (pin "1")
     (pin "2")
@@
       (effects (font (size 1.27 1.27)) hide)
     )
+    (property "dnp" "dnp" (id 4) (at 204.47 161.29 0)
+      (effects (font (size 1.27 1.27)) hide)
+    )
     (pin "1")
     (pin "2")
@@
     )
     (property "Datasheet" "~" (id 3) (at 204.47 153.67 0)
+      (effects (font (size 1.27 1.27)) hide)
+    )
+    (property "dnp" "dnp" (id 4) (at 204.47 153.67 0)
       (effects (font (size 1.27 1.27)) hide)
     )
@@
       (effects (font (size 1.27 1.27)) (justify left) hide)
     )
-    (property "Manufacturer_Name" "Phoenix Contact" (id 6) (at 262.89 124.46 0)
-      (effects (font (size 1.27 1.27)) (justify left) hide)
-    )
-    (property "Manufacturer_Part_Number" "1848668" (id 7) (at 262.89 127 0)
-      (effects (font (size 1.27 1.27)) (justify left) hide)
-    )
-    (property "Mouser Part Number" "651-1848668" (id 8) (at 262.89 129.54 0)
+    (property "Manufacturer_Name" "" (id 6) (at 262.89 124.46 0)
+      (effects (font (size 1.27 1.27)) (justify left) hide)
+    )
+    (property "Manufacturer_Part_Number" "" (id 7) (at 262.89 127 0)
+      (effects (font (size 1.27 1.27)) (justify left) hide)
+    )
+    (property "Mouser Part Number" "" (id 8) (at 262.89 129.54 0)
       (effects (font (size 1.27 1.27)) (justify left) hide)
     )
@@
     )
     (property "Manufacturer #" "1848668" (id 13) (at 241.3 116.84 0)
+      (effects (font (size 1.27 1.27)) hide)
+    )
+    (property "Mouser #" "651-1848668" (id 14) (at 241.3 116.84 0)
       (effects (font (size 1.27 1.27)) hide)
     )
@@
       (effects (font (size 1.27 1.27)) (justify left) hide)
     )
-    (property "Description" "Push spring connector 5mm pitch 8 way Phoenix Contact SDC Series 5mm Pitch Straight Pluggable Terminal Block, Plug with Plug In Termination, PCB Mount, 8 Way" (id 4) (at 257.81 26.67 0)
+    (property "Description" "Pluggable Terminal Blocks SDDC 1,5/ 4-PV-3,5" (id 4) (at 257.81 26.67 0)
       (effects (font (size 1.27 1.27)) (justify left) hide)
     )
@@
       (effects (font (size 1.27 1.27)) (justify left) hide)
     )
-    (property "Manufacturer_Name" "Phoenix Contact" (id 6) (at 257.81 31.75 0)
-      (effects (font (size 1.27 1.27)) (justify left) hide)
-    )
-    (property "Manufacturer_Part_Number" "1864095" (id 7) (at 257.81 34.29 0)
-      (effects (font (size 1.27 1.27)) (justify left) hide)
-    )
-    (property "Mouser Part Number" "651-1864095" (id 8) (at 257.81 36.83 0)
+    (property "Manufacturer_Name" "" (id 6) (at 257.81 31.75 0)
+      (effects (font (size 1.27 1.27)) (justify left) hide)
+    )
+    (property "Manufacturer_Part_Number" "" (id 7) (at 257.81 34.29 0)
+      (effects (font (size 1.27 1.27)) (justify left) hide)
+    )
+    (property "Mouser Part Number" "" (id 8) (at 257.81 36.83 0)
       (effects (font (size 1.27 1.27)) (justify left) hide)
     )
@@
     )
     (property "Manufacturer #" "1864095" (id 13) (at 241.3 24.13 0)
+      (effects (font (size 1.27 1.27)) hide)
+    )
+    (property "Mouser #" "651-1864095" (id 14) (at 241.3 24.13 0)
       (effects (font (size 1.27 1.27)) hide)
     )
@@
       (effects (font (size 1.27 1.27)) hide)
     )
+    (property "dnp" "dnp" (id 4) (at 204.47 146.05 0)
+      (effects (font (size 1.27 1.27)) hide)
+    )
     (pin "1")
     (pin "2")
@@
       (effects (font (size 1.27 1.27)) (justify left) hide)
     )
-    (property "Manufacturer_Name" "Phoenix Contact" (id 6) (at 262.89 148.59 0)
-      (effects (font (size 1.27 1.27)) (justify left) hide)
-    )
-    (property "Manufacturer_Part_Number" "1848668" (id 7) (at 262.89 151.13 0)
-      (effects (font (size 1.27 1.27)) (justify left) hide)
-    )
-    (property "Mouser Part Number" "651-1848668" (id 8) (at 262.89 153.67 0)
+    (property "Manufacturer_Name" "" (id 6) (at 262.89 148.59 0)
+      (effects (font (size 1.27 1.27)) (justify left) hide)
+    )
+    (property "Manufacturer_Part_Number" "" (id 7) (at 262.89 151.13 0)
+      (effects (font (size 1.27 1.27)) (justify left) hide)
+    )
+    (property "Mouser Part Number" "" (id 8) (at 262.89 153.67 0)
       (effects (font (size 1.27 1.27)) (justify left) hide)
     )
@@
     )
     (property "Manufacturer #" "1848668" (id 13) (at 241.3 140.97 0)
+      (effects (font (size 1.27 1.27)) hide)
+    )
+    (property "Mouser #" "651-1848668" (id 14) (at 241.3 140.97 0)
       (effects (font (size 1.27 1.27)) hide)
     )
@@
       (effects (font (size 1.27 1.27)) hide)
     )
+    (property "dnp" "dnp" (id 4) (at 204.47 148.59 0)
+      (effects (font (size 1.27 1.27)) hide)
+    )
     (pin "1")
     (pin "2")
@@
       (effects (font (size 1.27 1.27)) (justify left) hide)
     )
-    (property "Manufacturer_Name" "Phoenix Contact" (id 6) (at 262.89 77.47 0)
-      (effects (font (size 1.27 1.27)) (justify left) hide)
-    )
-    (property "Manufacturer_Part_Number" "1848668" (id 7) (at 262.89 80.01 0)
-      (effects (font (size 1.27 1.27)) (justify left) hide)
-    )
-    (property "Mouser Part Number" "651-1848668" (id 8) (at 262.89 82.55 0)
+    (property "Manufacturer_Name" "" (id 6) (at 262.89 77.47 0)
+      (effects (font (size 1.27 1.27)) (justify left) hide)
+    )
+    (property "Manufacturer_Part_Number" "" (id 7) (at 262.89 80.01 0)
+      (effects (font (size 1.27 1.27)) (justify left) hide)
+    )
+    (property "Mouser Part Number" "" (id 8) (at 262.89 82.55 0)
       (effects (font (size 1.27 1.27)) (justify left) hide)
     )
@@
       (effects (font (size 1.27 1.27)) hide)
     )
+    (property "Mouser #" "651-1848668" (id 14) (at 241.3 69.85 0)
+      (effects (font (size 1.27 1.27)) hide)
+    )

Commit message: changes
Parts:
- removed J10: Ch 5-8, Component Search Engine:Pluggable Terminal Blocks SDDC 1.5mm pitch 8 Pin, symbol Component Search Engine:Pluggable Terminal Blocks SDDC 1.5mm pitch 8 Pin
- removed J11: Ch 9-12, Component Search Engine:Pluggable Terminal Blocks SDDC 1.5mm pitch 8 Pin, symbol Component Search Engine:Pluggable Terminal Blocks SDDC 1.5mm pitch 8 Pin
- removed NT1, NT2, NT3, NT4, NT5, NT6, NT7, NT8: NetTie_2, NetTie:NetTie-2_SMD_Pad0.5mm, symbol Device:NetTie_2
- added J10, J11: Ch 1-4, Component Search Engine:Pluggable Terminal Blocks SDC 2.5mm pitch 8 Pin, symbol Component Search Engine:Pluggable Terminal Blocks SDC 2.5mm pitch 8 Pin
Connections:
- net I/O Ch10 High: now also J11.4
- net I/O Ch10 Low: now also J11.3
- net I/O Ch11 High: now also J11.6
- net I/O Ch11 Low: now also J11.5
- net I/O Ch12 High: now also J11.8
- net I/O Ch12 Low: now also J11.7
- net I/O Ch5 High: now also J10.2
- net I/O Ch5 Low: now also J10.1
- net I/O Ch6 High: now also J10.4
- net I/O Ch6 Low: now also J10.3
- net I/O Ch7 High: now also J10.6
- net I/O Ch7 Low: now also J10.5
- net I/O Ch8 High: now also J10.8
- net I/O Ch8 Low: now also J10.7
- net I/O Ch9 High: now also J11.2
- net I/O Ch9 Low: now also J11.1
Other:
- note removed: "Net-ties are used to change net size"
