File: CIB_Main_PCB - Mimic Octopus/DUT Power.kicad_sch (KiCad schematic)
At the start: 37 parts, among them K18 PC357, K19 PC357, U1 HMSR_30-SMS, U2 HMSR_30-SMS

Commit message: message
Parts:
- D24: footprint (none) -> Diode_SMD:D_SMB_Handsoldering
Changed lines of the file:
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@@
       (effects (font (size 1.27 1.27)) (justify left))
     )
-    (property "Footprint" "" (id 2) (at 255.27 34.29 90)
+    (property "Footprint" "Diode_SMD:D_SMB_Handsoldering" (id 2) (at 255.27 34.29 90)
       (effects (font (size 1.27 1.27)) hide)
     )

Commit message: added changes
Parts:
- U1, U2: footprint LEM_Current_Transducer_HMSR-SMS:HMSR-SMS -> Component Search Engine:HMSR6SMS
- renumbered C4 to C1, C8 to C10, C5 to C2, C6 to C3, C15 to C4, C16 to C5, C9 to C6, C10 to C7, C17 to C8, C7 to C9, D24 to D1, D15 to D2, D25 to D3, D16 to D4, D9 to D5, K9 to K1, K18 to K2, K10 to K3, K19 to K4, R29 to R11, R30 to R12, R14 to R13, R45 to R14, R32 to R15, R33 to R16, R34 to R17, R35 to R18, R36 to R19, R16 to R20, R37 to R21, R38 to R22, R39 to R23, R53 to R24, R13 to R25, R15 to R26

Commit message: V0.1 PCB to be sent out
Parts:
- added NT9: NetTie_2, NetTie:NetTie-2_SMD_Pad0.5mm, symbol Device:NetTie_2
- added R171: 1k2, Resistor_SMD:R_1206_3216Metric_Pad1.30x1.75mm_HandSolder, symbol Device:R_Small
Connections:
- net DUT Power Ch1: now also NT9.2; no longer R25.1
- net DUT Supply V monitor: now also R171.2; no longer C10.1, C9.1, D5.1 (K), D5.2 (K), R25.2, R26.1
- new net: NT9.1, R25.1
- new net: C10.1, C9.1, D5.1 (K), D5.2 (K), R171.1, R25.2, R26.1
Changed lines of the file:
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@@
   (junction (at 255.27 82.55) (diameter 0) (color 0 0 0 0)
   )
+  (junction (at 34.29 39.37) (diameter 0) (color 0 0 0 0)
+  )
   (junction (at 74.93 175.26) (diameter 0) (color 0 0 0 0)
   )
-  (junction (at 34.29 39.37) (diameter 0) (color 0 0 0 0)
-  )
   (junction (at 247.65 41.91) (diameter 0) (color 0 0 0 0)
   )
@@
     (stroke (width 0) (type default) (color 0 0 0 0))
   )
-  (wire (pts (xy 33.02 166.37) (xy 33.02 167.64))
-    (stroke (width 0) (type default) (color 0 0 0 0))
-  )
   (wire (pts (xy 247.65 97.79) (xy 243.84 97.79))
     (stroke (width 0) (type default) (color 0 0 0 0))
@@
     (stroke (width 0) (type default) (color 0 0 0 0))
   )
-  (wire (pts (xy 77.47 175.26) (xy 74.93 175.26))
-    (stroke (width 0) (type default) (color 0 0 0 0))
-  )
   (wire (pts (xy 255.27 97.79) (xy 247.65 97.79))
     (stroke (width 0) (type default) (color 0 0 0 0))
@@
     (stroke (width 0) (type default) (color 0 0 0 0))
   )
+  (wire (pts (xy 74.93 175.26) (xy 77.47 175.26))
+    (stroke (width 0) (type default) (color 0 0 0 0))
+  )
   (wire (pts (xy 111.76 90.17) (xy 121.92 90.17))
     (stroke (width 0) (type default) (color 0 0 0 0))
@@
   )
   (text "Vout =    Rbottom      * Vin\n	   ----------\n       Rtop + Rbottom\n\nVout	= 0-5 VDC\n12 VDC	= 0-18 VDC (under fault conditions)"
-    (at 44.45 170.18 0)
+    (at 43.18 166.37 0)
     (effects (font (size 1.27 1.27)) (justify left bottom))
   )
@@
     (effects (font (size 1.27 1.27)) (justify right bottom))
   )
-  (label "DUT Power Ch1" (at 33.02 166.37 180)
+  (label "DUT Power Ch1" (at 33.02 162.56 180)
     (effects (font (size 1.27 1.27)) (justify right bottom))
   )
@@
     (effects (font (size 1.27 1.27)) (justify left))
   )
-  (hierarchical_label "DUT Supply V monitor" (shape output) (at 77.47 175.26 0)
+  (hierarchical_label "DUT Supply V monitor" (shape output) (at 82.55 175.26 0)
     (effects (font (size 1.27 1.27)) (justify left))
   )
@@
     (pin "2")
   )
+  (symbol (lib_id "Device:R_Small") (at 80.01 175.26 90) (unit 1)
+    (in_bom yes) (on_board yes) (fields_autoplaced)
+    (property "Reference" "R171" (id 0) (at 80.01 168.91 90))
+    (property "Value" "1k2" (id 1) (at 80.01 171.45 90))
+    (property "Footprint" "Resistor_SMD:R_1206_3216Metric_Pad1.30x1.75mm_HandSolder" (id 2) (at 80.01 175.26 0)
+      (effects (font (size 1.27 1.27)) hide)
+    )
+    (property "Datasheet" "https://industrial.panasonic.com/ww/products/pt/general-purpose-chip-resistors/models/ERJ6GEYJ681V" (id 3) (at 80.01 175.26 0)
+      (effects (font (size 1.27 1.27)) hide)
+    )
+    (property "DigiKey #" "P2.0KACT-ND" (id 4) (at 80.01 175.26 0)
+      (effects (font (size 1.27 1.27)) hide)
+    )
+    (property "Manufacturer #" "ERJ-6GEYJ202V" (id 5) (at 80.01 175.26 0)
+      (effects (font (size 1.27 1.27)) hide)
+    )
+    (property "Manufacturer" "Panasonic Electronics Company" (id 6) (at 80.01 175.26 0)
+      (effects (font (size 1.27 1.27)) hide)
+    )
+    (property "Farnell #" "2057707" (id 7) (at 80.01 175.26 0)
+      (effects (font (size 1.27 1.27)) hide)
+    )
+    (pin "1")
+    (pin "2")
+  )
   (symbol (lib_id "Device:D_Schottky_KKA") (at 72.39 181.61 270) (unit 1)
     (in_bom yes) (on_board yes) (fields_autoplaced)
@@
       (effects (font (size 1.27 1.27)) hide)
     )
+    (pin "1")
+    (pin "2")
+  )
+  (symbol (lib_id "Device:NetTie_2") (at 33.02 165.1 90) (unit 1)
+    (in_bom yes) (on_board yes) (fields_autoplaced)
+    (property "Reference" "NT9" (id 0) (at 27.94 165.1 0)
+      (effects (font (size 1.27 1.27)) hide)
+    )
+    (property "Value" "NetTie_2" (id 1) (at 30.48 165.1 0)
+      (effects (font (size 1.27 1.27)) hide)
+    )
+    (property "Footprint" "NetTie:NetTie-2_SMD_Pad0.5mm" (id 2) (at 33.02 165.1 0)
+      (effects (font (size 1.27 1.27)) hide)
+    )
+    (property "Datasheet" "~" (id 3) (at 33.02 165.1 0)
+      (effects (font (size 1.27 1.27)) hide)
+    )

Commit message: BoM
Parts:
- C1, C4, C5, C8: value 100nF 60V -> 0.1uF 63V; DigiKey # 1276-1137-1-ND -> 399-C1206C104MMREC7210CT-ND; DigiKey Price/Stock https://www.digikey.co.uk/en/products/detail/samsung-electr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 -> https://www.digikey.co.uk/en/products/detail/kemet/C1206C10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; Height (none) -> 2; Manufacturer Samsung Electro-Mechanics -> Kemet; Manufacturer # CL31A106KOHNNNE -> C1206C104MMREC7210
- C10: DigiKey # 732-7642-1-ND -> 1276-3048-1-ND; DigiKey Price/Stock https://www.digikey.co.uk/en/products/detail/w%C3%BCrth-ele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 -> https://www.digikey.co.uk/en/products/detail/samsung-electr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; Height (none) -> 2; Manufacturer Würth Elektronik -> Samsung Electro-Mechanics; Manufacturer # 885012108018 -> CL31A226KOHNNNE
- C2, C3, C6, C7, C9, D5: Height (none) -> 2
- D1, D3: value 55V -> 56V; DigiKey # (none) -> 641-1818-1-ND; DigiKey Price/Stock (none) -> https://www.digikey.co.uk/en/products/detail/comchip-techno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; Height (none) -> 3; Manufacturer (none) -> Comchip Technology; Manufacturer # (none) -> CZRB5370B-HF
- D2, D4: DigiKey Price/Stock (none) -> https://www.digikey.co.uk/en/products/detail/w%C3%BCrth-ele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; Height (none) -> 2
- K1, K3: DigiKey Price/Stock (none) -> https://www.digikey.co.uk/en/products/detail/finder-relays-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; Manufacturer (none) -> Finder Relays, Inc
- K2, K4: DigiKey Price/Stock (none) -> https://www.digikey.co.uk/en/products/detail/picker-compone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
- NT9: dnp (none) -> dnp
- R11, R13, R16, R18, R20, R23: DigiKey # (none) -> 13-RC1206JR-7W0RLCT-ND; DigiKey Price/Stock (none) -> https://www.digikey.co.uk/en/products/detail/yageo/RC1206JR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; Farnell # 2861314 -> (none); Manufacturer TE Connectivity -> Yago; Manufacturer # CRGP2010F1M0 -> RC1206JR-7W0RL
- R12, R15, R19, R22: dnp dnp -> (none)

Commit message: changes
Parts:
- removed D2, D4: Green, Diode_SMD:D_1206_3216Metric_Pad1.42x1.75mm_HandSolder, symbol Device:LED_Small_Filled
- removed R17, R24: 1k2, Resistor_SMD:R_1206_3216Metric_Pad1.30x1.75mm_HandSolder, symbol Device:R_Small
- added J2: DUT Power Out, Component Search Engine:Pluggable Terminal Blocks SDC 2.5mm pitch 12 Pin, symbol Component Search Engine:Pluggable Terminal Blocks SDC 2,5/12-PV-5,0 0-ZB
- K1, K3: value ~ -> 30A
- NT9: value NetTie_2 -> NetTie
Connections:
- net DUT Power 1 +VE: now also J2.1, J2.3, J2.5
- net DUT Power 1 -VE: now also J2.2, J2.4, J2.6
- net DUT Power 2 +VE: now also J2.11, J2.7, J2.9
- net DUT Power 2 -VE: now also J2.10, J2.12, J2.8
