File: CIB_Main_PCB - Mimic Octopus/External Equipment Connections.kicad_sch (KiCad schematic)
At the start: 45 parts, among them J12 External Equipment, U29 HMSR_8-SMS, U30 HMSR_8-SMS, U31 HMSR_8-SMS, U32 HMSR_8-SMS

Commit message: message
Parts:
- R23, R24, R46, R47: dnp (none) -> dnp
Connections:
- net Eq Ch1 Low: now also R41.1, R46.2
- net Eq Ch2 Low: now also R23.2, R42.1
- net Eq Ch3 Low: now also R24.2, R43.1
- net Eq Ch4 Low: now also R44.1, R47.2
Other:
- note removed: "Vout = Rbottom * Vin ---------- Rtop + Rbottom Vout = 0-10 VDC Vin = 0-52 VDC"
- moved on the sheet: R23, R24, R41, R42, R43, R44, R46, R47

Commit message: added changes
Parts:
- J15: renamed from J12; footprint Component Search Engine:Pluggable Terminal Blocks SDC 2,5 12-PV-5,0 0-ZB -> Component Search Engine:Pluggable Terminal Blocks SDC 2.5mm pitch 12 Pin
- U31: renamed from U29; footprint LEM_Current_Transducer_HMSR-SMS:HMSR-SMS -> Component Search Engine:HMSR6SMS
- U32: renamed from U30; footprint LEM_Current_Transducer_HMSR-SMS:HMSR-SMS -> Component Search Engine:HMSR6SMS
- U33: renamed from U31; footprint LEM_Current_Transducer_HMSR-SMS:HMSR-SMS -> Component Search Engine:HMSR6SMS
- U34: renamed from U32; footprint LEM_Current_Transducer_HMSR-SMS:HMSR-SMS -> Component Search Engine:HMSR6SMS
- renumbered C52 to C56, C53 to C57, C54 to C58, C55 to C59, C56 to C60, C57 to C61, C58 to C62, C59 to C63, C60 to C64, C61 to C65, C62 to C66, C63 to C67, C64 to C68, C65 to C69, C66 to C70, C67 to C71, D77 to D60, D78 to D61, D79 to D62, D80 to D63, R46 to R100, R23 to R101, R24 to R102, R47 to R103, R143 to R104, R49 to R105, R144 to R106, R137 to R87, R21 to R88, R138 to R89, R139 to R90, R22 to R91, R140 to R92, R141 to R93, R48 to R94, R142 to R95, R41 to R96, R42 to R97, R43 to R98, R44 to R99

Commit message: V0.1 PCB to be sent out
Parts:
- added NT10, NT11, NT12, NT13: NetTie_2, NetTie:NetTie-2_SMD_Pad0.5mm, symbol Device:NetTie_2
- added R172, R173, R174, R175: 1k2, Resistor_SMD:R_1206_3216Metric_Pad1.30x1.75mm_HandSolder, symbol Device:R_Small
Connections:
- net Eq Ch1 High: now also NT10.1; no longer R87.1
- net Eq Ch1 V monitor: now also R172.2; no longer C57.1, C58.1, D60.1 (K), D60.2 (K), R87.2, R89.1
- net Eq Ch2 High: now also NT11.1; no longer R90.1
- net Eq Ch2 V monitor: now also R173.2; no longer C61.1, C62.1, D61.1 (K), D61.2 (K), R90.2, R92.1
- net Eq Ch3 High: now also NT12.1; no longer R93.1
- net Eq Ch3 V monitor: now also R174.2; no longer C65.1, C66.1, D62.1 (K), D62.2 (K), R93.2, R95.1
- net Eq Ch4 High: now also NT13.1; no longer R104.1
- net Eq Ch4 V monitor: now also R175.2; no longer C69.1, C70.1, D63.1 (K), D63.2 (K), R104.2, R106.1
- new net: NT11.2, R90.1
- new net: C61.1, C62.1, D61.1 (K), D61.2 (K), R173.1, R90.2, R92.1
- new net: NT10.2, R87.1
- new net: C69.1, C70.1, D63.1 (K), D63.2 (K), R104.2, R106.1, R175.1
- new net: NT13.2, R104.1
- new net: C57.1, C58.1, D60.1 (K), D60.2 (K), R172.1, R87.2, R89.1
- new net: NT12.2, R93.1
- new net: C65.1, C66.1, D62.1 (K), D62.2 (K), R174.1, R93.2, R95.1

Commit message: BoM
Parts:
- C56, C57, C59, C60, C61, C63, C64, C65, C67, C68, C69, C71, D60, D61, D62, D63: Height (none) -> 2
- C58, C62, C66, C70: DigiKey # 732-7642-1-ND -> 1276-3048-1-ND; DigiKey Price/Stock https://www.digikey.co.uk/en/products/detail/w%C3%BCrth-ele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 -> https://www.digikey.co.uk/en/products/detail/samsung-electr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; Height (none) -> 2; Manufacturer Würth Elektronik -> Samsung Electro-Mechanics; Manufacturer # 885012108018 -> CL31A226KOHNNNE
- J15: Mouser # (none) -> 651-1864134; Mouser Part Number 651-1864134 -> (none)
- NT10, NT11, NT12, NT13: dnp (none) -> dnp
- R100, R101, R102, R103, R105, R88, R91, R94: DigiKey # YAG3380DKR-ND -> 13-RC1206JR-7W0RLCT-ND; DigiKey Price/Stock (none) -> https://www.digikey.co.uk/en/products/detail/yageo/RC1206JR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; Farnell # 9235523 -> (none); Manufacturer YAGEO -> Yago; Manufacturer # RC2010JK-070RL -> RC1206JR-7W0RL
- U31, U32, U33, U34: Height (none) -> 5

Commit message: changes
Parts:
- NT10, NT11, NT12, NT13: value NetTie_2 -> NetTie
Changed lines of the file:
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@@
   (symbol (lib_id "Device:R_Small") (at 218.44 129.54 180) (unit 1)
     (in_bom yes) (on_board yes) (fields_autoplaced)
-    (property "Reference" "R101" (id 0) (at 215.9 126.9999 0)
-      (effects (font (size 1.27 1.27)) (justify left))
-    )
-    (property "Value" "0" (id 1) (at 215.9 129.5399 0)
-      (effects (font (size 1.27 1.27)) (justify left))
+    (property "Reference" "R101" (id 0) (at 220.98 126.9999 0)
+      (effects (font (size 1.27 1.27)) (justify right))
+    )
+    (property "Value" "0" (id 1) (at 220.98 129.5399 0)
+      (effects (font (size 1.27 1.27)) (justify right))
     )
     (property "Footprint" "Resistor_SMD:R_2010_5025Metric_Pad1.40x2.65mm_HandSolder" (id 2) (at 218.44 129.54 0)
@@
       (effects (font (size 1.27 1.27)) hide)
     )
-    (property "dnp" "dnp" (id 11) (at 215.9 132.0799 0)
-      (effects (font (size 1.27 1.27)) (justify left))
+    (property "dnp" "dnp" (id 11) (at 220.98 132.0799 0)
+      (effects (font (size 1.27 1.27)) (justify right))
     )
     (property "Description" "0 Ohms Jumper 0.5W, 1/2W Chip Resistor 1206 (3216 Metric) Moisture Resistant Thick Film" (id 12) (at 218.44 129.54 0)
@@
       (effects (font (size 1.27 1.27)) hide)
     )
-    (property "Value" "NetTie_2" (id 1) (at 119.38 17.78 0)
+    (property "Value" "NetTie" (id 1) (at 119.38 17.78 0)
       (effects (font (size 1.27 1.27)) hide)
     )
@@
       (effects (font (size 1.27 1.27)) hide)
     )
-    (property "Value" "NetTie_2" (id 1) (at 119.38 149.86 0)
+    (property "Value" "NetTie" (id 1) (at 119.38 149.86 0)
       (effects (font (size 1.27 1.27)) hide)
     )
@@
       (effects (font (size 1.27 1.27)) hide)
     )
-    (property "Value" "NetTie_2" (id 1) (at 119.38 60.96 0)
+    (property "Value" "NetTie" (id 1) (at 119.38 60.96 0)
       (effects (font (size 1.27 1.27)) hide)
     )
@@
   (symbol (lib_id "Device:D_Schottky_KKA") (at 161.29 168.91 270) (unit 1)
     (in_bom yes) (on_board yes) (fields_autoplaced)
-    (property "Reference" "D63" (id 0) (at 163.83 167.6399 90)
-      (effects (font (size 1.27 1.27)) (justify left))
-    )
-    (property "Value" "5V1" (id 1) (at 163.83 170.1799 90)
+    (property "Reference" "D63" (id 0) (at 165.1 166.3699 90)
+      (effects (font (size 1.27 1.27)) (justify left))
+    )
+    (property "Value" "5V1" (id 1) (at 165.1 168.9099 90)
       (effects (font (size 1.27 1.27)) (justify left))
     )
@@
       (effects (font (size 1.27 1.27)) hide)
     )
-    (property "Value" "NetTie_2" (id 1) (at 119.38 102.87 0)
+    (property "Value" "NetTie" (id 1) (at 119.38 102.87 0)
       (effects (font (size 1.27 1.27)) hide)
     )
@@
   (symbol (lib_id "Device:D_Schottky_KKA") (at 161.29 80.01 270) (unit 1)
     (in_bom yes) (on_board yes) (fields_autoplaced)
-    (property "Reference" "D61" (id 0) (at 163.83 78.7399 90)
-      (effects (font (size 1.27 1.27)) (justify left))
-    )
-    (property "Value" "5V1" (id 1) (at 163.83 81.2799 90)
+    (property "Reference" "D61" (id 0) (at 165.1 77.4699 90)
+      (effects (font (size 1.27 1.27)) (justify left))
+    )
+    (property "Value" "5V1" (id 1) (at 165.1 80.0099 90)
       (effects (font (size 1.27 1.27)) (justify left))
     )
@@
   (symbol (lib_id "Device:R_Small") (at 227.33 129.54 180) (unit 1)
     (in_bom yes) (on_board yes) (fields_autoplaced)
-    (property "Reference" "R102" (id 0) (at 224.79 126.9999 0)
-      (effects (font (size 1.27 1.27)) (justify left))
-    )
-    (property "Value" "0" (id 1) (at 224.79 129.5399 0)
-      (effects (font (size 1.27 1.27)) (justify left))
+    (property "Reference" "R102" (id 0) (at 229.87 126.9999 0)
+      (effects (font (size 1.27 1.27)) (justify right))
+    )
+    (property "Value" "0" (id 1) (at 229.87 129.5399 0)
+      (effects (font (size 1.27 1.27)) (justify right))
     )
     (property "Footprint" "Resistor_SMD:R_2010_5025Metric_Pad1.40x2.65mm_HandSolder" (id 2) (at 227.33 129.54 0)
@@
       (effects (font (size 1.27 1.27)) hide)
     )
-    (property "dnp" "dnp" (id 11) (at 224.79 132.0799 0)
-      (effects (font (size 1.27 1.27)) (justify left))
+    (property "dnp" "dnp" (id 11) (at 229.87 132.0799 0)
+      (effects (font (size 1.27 1.27)) (justify right))
     )
     (property "Description" "0 Ohms Jumper 0.5W, 1/2W Chip Resistor 1206 (3216 Metric) Moisture Resistant Thick Film" (id 12) (at 227.33 129.54 0)
@@
   (symbol (lib_id "Device:R_Small") (at 236.22 129.54 180) (unit 1)
     (in_bom yes) (on_board yes) (fields_autoplaced)
-    (property "Reference" "R103" (id 0) (at 233.68 126.9999 0)
-      (effects (font (size 1.27 1.27)) (justify left))
-    )
-    (property "Value" "0" (id 1) (at 233.68 129.5399 0)
-      (effects (font (size 1.27 1.27)) (justify left))
+    (property "Reference" "R103" (id 0) (at 238.76 126.9999 0)
+      (effects (font (size 1.27 1.27)) (justify right))
+    )
+    (property "Value" "0" (id 1) (at 238.76 129.5399 0)
+      (effects (font (size 1.27 1.27)) (justify right))
     )
     (property "Footprint" "Resistor_SMD:R_2010_5025Metric_Pad1.40x2.65mm_HandSolder" (id 2) (at 236.22 129.54 0)
@@
       (effects (font (size 1.27 1.27)) hide)
     )
-    (property "dnp" "dnp" (id 11) (at 233.68 132.0799 0)
-      (effects (font (size 1.27 1.27)) (justify left))
+    (property "dnp" "dnp" (id 11) (at 238.76 132.0799 0)
+      (effects (font (size 1.27 1.27)) (justify right))
     )
     (property "Description" "0 Ohms Jumper 0.5W, 1/2W Chip Resistor 1206 (3216 Metric) Moisture Resistant Thick Film" (id 12) (at 236.22 129.54 0)
@@
   (symbol (lib_id "Device:D_Schottky_KKA") (at 161.29 36.83 270) (unit 1)
     (in_bom yes) (on_board yes) (fields_autoplaced)
-    (property "Reference" "D60" (id 0) (at 163.83 35.5599 90)
-      (effects (font (size 1.27 1.27)) (justify left))
-    )
-    (property "Value" "5V1" (id 1) (at 163.83 38.0999 90)
+    (property "Reference" "D60" (id 0) (at 165.1 34.2899 90)
+      (effects (font (size 1.27 1.27)) (justify left))
+    )
+    (property "Value" "5V1" (id 1) (at 165.1 36.8299 90)
       (effects (font (size 1.27 1.27)) (justify left))
     )
@@
   (symbol (lib_id "Device:D_Schottky_KKA") (at 161.29 121.92 270) (unit 1)
     (in_bom yes) (on_board yes) (fields_autoplaced)
-    (property "Reference" "D62" (id 0) (at 163.83 120.6499 90)
-      (effects (font (size 1.27 1.27)) (justify left))
-    )
-    (property "Value" "5V1" (id 1) (at 163.83 123.1899 90)
-      (effects (font (size 1.27 1.27)) (justify left))
-    )
+    (property "Reference" "D62" (id 0) (at 165.1 119.3799 90)
+      (effects (font (size 1.27 1.27)) (justify left))
+    )
+    (property "Value" "5V1" (id 1) (at 165.1 121.9199 90)
+      (effects (font (size 1.27 1.27)) (justify left))
+    )
