File: CIB_Main_PCB - Mimic Octopus/PT100 PT1000 Simulation.kicad_sch (KiCad schematic)
At the start: 19 parts, among them J17 PT1-4

Commit message: added changes
Parts:
- J8: renamed from J17; footprint Component Search Engine:Pluggable Terminal Blocks SDDC 1,5 4-PV-3,5 -> Component Search Engine:Pluggable Terminal Blocks SDDC 1.5mm pitch 8 Pin; symbol Component Search Engine:Pluggable Terminal Blocks SDDC 1,5/ 4-PV-3,5 -> Component Search Engine:Pluggable Terminal Blocks SDDC 1.5mm pitch 8 Pin; Manufacturer_Name (none) -> Phoenix Contact; Manufacturer_Part_Number (none) -> 1848668
- renumbered D12 to D14, D13 to D15, D14 to D16, D10 to D17, D11 to D18, K12 to K13, K13 to K14, K14 to K15, K15 to K16, K11 to K17, R25 to R35, R26 to R36, R27 to R37, R19 to R38, R20 to R39, R31 to R40, R17 to R41, R18 to R42

Commit message: BoM
Parts:
- D14, D15, D16, D17, D18: DigiKey Price/Stock (none) -> https://www.digikey.co.uk/en/products/detail/w%C3%BCrth-ele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; Height (none) -> 2
- J8: Manufacturer_Name Phoenix Contact -> (none); Manufacturer_Part_Number 1848668 -> (none); Mouser # (none) -> 651-1848668; Mouser Part Number 651-1848668 -> (none)
- K13, K14, K15, K16, K17: value ~ -> G6K-2P DC12; DigiKey Price/Stock (none) -> https://www.digikey.co.uk/en/products/detail/omron-electron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; Manufacture Omron Electronics Inc-EMC Div -> (none); Manufacturer (none) -> Omron Electronics Inc-EMC Div
- R36: Mouser # (none) -> 667-ERA-8AEB1020V; Mouser Part Number 667-ERA-8AEB1020V -> (none)
- R37: Mouser # (none) -> 667-ERA-8AEB1150V; Mouser Part Number 667-ERA-8AEB1150V -> (none)

Commit message: changes
Parts:
- removed D14, D15, D16, D17, D18: Green, Diode_SMD:D_1206_3216Metric_Pad1.42x1.75mm_HandSolder, symbol Device:LED_Small_Filled
- removed R38, R39, R40, R41, R42: 1k2, Resistor_SMD:R_1206_3216Metric_Pad1.30x1.75mm_HandSolder, symbol Device:R_Small
- K13, K14, K15, K16, K17: value G6K-2P DC12 -> PC357; footprint Relay_THT:Relay_DPDT_Omron_G6K-2P -> _Connectors:PC375; DigiKey # Z117-ND -> 2634-PC375-2C-12S4-X-ND; DigiKey Price/Stock https://www.digikey.co.uk/en/products/detail/omron-electron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 -> https://www.digikey.co.uk/en/products/detail/picker-compone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; Manufacturer Omron Electronics Inc-EMC Div -> Picker Components; Manufacturer # G6K-2P DC12 -> PC375-2C-12S4-X
