File: CIB_Main_PCB - Mimic Octopus/RAG.kicad_sch (KiCad schematic)
At the start: 12 parts

Commit message: added changes
Parts:
- renumbered D17 to D55, D18 to D56, D20 to D57, D21 to D58, D22 to D59, K16 to K50, K17 to K51, R79 to R82, R80 to R83, R81 to R84, R82 to R85, R83 to R86
Changed lines of the file:
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@@
   (symbol (lib_id "Device:R_Small") (at 166.37 93.98 0) (unit 1)
     (in_bom yes) (on_board yes) (fields_autoplaced)
-    (property "Reference" "R79" (id 0) (at 168.91 92.7099 0)
+    (property "Reference" "R82" (id 0) (at 168.91 92.7099 0)
       (effects (font (size 1.27 1.27)) (justify left))
     )
@@
   (symbol (lib_id "Device:LED_Small_Filled") (at 166.37 101.6 90) (unit 1)
     (in_bom yes) (on_board yes) (fields_autoplaced)
-    (property "Reference" "D17" (id 0) (at 168.91 100.2664 90)
+    (property "Reference" "D55" (id 0) (at 168.91 100.2664 90)
       (effects (font (size 1.27 1.27)) (justify right))
     )
@@
   (symbol (lib_id "Device:R_Small") (at 143.51 105.41 90) (unit 1)
     (in_bom yes) (on_board yes) (fields_autoplaced)
-    (property "Reference" "R83" (id 0) (at 143.51 109.22 90))
+    (property "Reference" "R86" (id 0) (at 143.51 109.22 90))
     (property "Value" "1k2" (id 1) (at 143.51 111.76 90))
     (property "Footprint" "Resistor_SMD:R_1206_3216Metric_Pad1.30x1.75mm_HandSolder" (id 2) (at 143.51 105.41 0)
@@
   (symbol (lib_id "power:GND") (at 176.53 105.41 0) (unit 1)
     (in_bom yes) (on_board yes) (fields_autoplaced)
-    (property "Reference" "#PWR0413" (id 0) (at 176.53 111.76 0)
+    (property "Reference" "#PWR0252" (id 0) (at 176.53 111.76 0)
       (effects (font (size 1.27 1.27)) hide)
     )
@@
   (symbol (lib_id "Device:R_Small") (at 176.53 93.98 0) (unit 1)
     (in_bom yes) (on_board yes) (fields_autoplaced)
-    (property "Reference" "R80" (id 0) (at 179.07 92.7099 0)
+    (property "Reference" "R83" (id 0) (at 179.07 92.7099 0)
       (effects (font (size 1.27 1.27)) (justify left))
     )
@@
   (symbol (lib_id "Relay:G2RL-2-DC24") (at 106.68 86.36 270) (mirror x) (unit 1)
     (in_bom yes) (on_board yes) (fields_autoplaced)
-    (property "Reference" "K16" (id 0) (at 106.68 68.58 90))
+    (property "Reference" "K50" (id 0) (at 106.68 68.58 90))
     (property "Value" "~" (id 1) (at 106.68 68.072 90)
       (effects (font (size 1.27 1.27)) hide)
@@
   (symbol (lib_id "Device:R_Small") (at 186.69 93.98 0) (unit 1)
     (in_bom yes) (on_board yes) (fields_autoplaced)
-    (property "Reference" "R81" (id 0) (at 189.23 92.7099 0)
+    (property "Reference" "R84" (id 0) (at 189.23 92.7099 0)
       (effects (font (size 1.27 1.27)) (justify left))
     )
@@
   (symbol (lib_id "power:+12V") (at 139.7 96.52 0) (unit 1)
     (in_bom yes) (on_board yes) (fields_autoplaced)
-    (property "Reference" "#PWR0409" (id 0) (at 139.7 100.33 0)
+    (property "Reference" "#PWR0250" (id 0) (at 139.7 100.33 0)
       (effects (font (size 1.27 1.27)) hide)
     )
@@
   (symbol (lib_id "Device:LED_Small_Filled") (at 151.13 105.41 180) (unit 1)
     (in_bom yes) (on_board yes) (fields_autoplaced)
-    (property "Reference" "D22" (id 0) (at 151.0665 109.22 0))
+    (property "Reference" "D59" (id 0) (at 151.0665 109.22 0))
     (property "Value" "Green" (id 1) (at 151.0665 111.76 0))
     (property "Footprint" "Diode_SMD:D_1206_3216Metric_Pad1.42x1.75mm_HandSolder" (id 2) (at 151.13 105.41 90)
@@
   (symbol (lib_id "Device:LED_Small_Filled") (at 186.69 101.6 90) (unit 1)
     (in_bom yes) (on_board yes) (fields_autoplaced)
-    (property "Reference" "D20" (id 0) (at 189.23 100.2664 90)
+    (property "Reference" "D57" (id 0) (at 189.23 100.2664 90)
       (effects (font (size 1.27 1.27)) (justify right))
     )
@@
   (symbol (lib_id "Device:LED_Small_Filled") (at 110.49 105.41 180) (unit 1)
     (in_bom yes) (on_board yes) (fields_autoplaced)
-    (property "Reference" "D21" (id 0) (at 110.4265 109.22 0))
+    (property "Reference" "D58" (id 0) (at 110.4265 109.22 0))
     (property "Value" "Green" (id 1) (at 110.4265 111.76 0))
     (property "Footprint" "Diode_SMD:D_1206_3216Metric_Pad1.42x1.75mm_HandSolder" (id 2) (at 110.49 105.41 90)
@@
   (symbol (lib_id "power:+12V") (at 99.06 73.66 0) (unit 1)
     (in_bom yes) (on_board yes) (fields_autoplaced)
-    (property "Reference" "#PWR0410" (id 0) (at 99.06 77.47 0)
+    (property "Reference" "#PWR0248" (id 0) (at 99.06 77.47 0)
       (effects (font (size 1.27 1.27)) hide)
     )
@@
   (symbol (lib_id "power:+12V") (at 99.06 96.52 0) (unit 1)
     (in_bom yes) (on_board yes) (fields_autoplaced)
-    (property "Reference" "#PWR0411" (id 0) (at 99.06 100.33 0)
+    (property "Reference" "#PWR0249" (id 0) (at 99.06 100.33 0)
       (effects (font (size 1.27 1.27)) hide)
     )
@@
   (symbol (lib_id "Device:R_Small") (at 102.87 105.41 90) (unit 1)
     (in_bom yes) (on_board yes) (fields_autoplaced)
-    (property "Reference" "R82" (id 0) (at 102.87 109.22 90))
+    (property "Reference" "R85" (id 0) (at 102.87 109.22 90))
     (property "Value" "1k2" (id 1) (at 102.87 111.76 90))
     (property "Footprint" "Resistor_SMD:R_1206_3216Metric_Pad1.30x1.75mm_HandSolder" (id 2) (at 102.87 105.41 0)
@@
   (symbol (lib_id "Device:LED_Small_Filled") (at 176.53 101.6 90) (unit 1)
     (in_bom yes) (on_board yes) (fields_autoplaced)
-    (property "Reference" "D18" (id 0) (at 179.07 100.2664 90)
+    (property "Reference" "D56" (id 0) (at 179.07 100.2664 90)
       (effects (font (size 1.27 1.27)) (justify right))
     )
@@
   (symbol (lib_id "power:GND") (at 166.37 105.41 0) (unit 1)
     (in_bom yes) (on_board yes) (fields_autoplaced)
-    (property "Reference" "#PWR0414" (id 0) (at 166.37 111.76 0)
+    (property "Reference" "#PWR0251" (id 0) (at 166.37 111.76 0)
       (effects (font (size 1.27 1.27)) hide)
     )
@@
   (symbol (lib_id "Relay:G2RL-2-DC24") (at 147.32 86.36 270) (mirror x) (unit 1)
     (in_bom yes) (on_board yes) (fields_autoplaced)
-    (property "Reference" "K17" (id 0) (at 147.32 68.58 90))
+    (property "Reference" "K51" (id 0) (at 147.32 68.58 90))
     (property "Value" "~" (id 1) (at 147.32 68.072 90)
       (effects (font (size 1.27 1.27)) hide)
@@
   (symbol (lib_id "power:GND") (at 186.69 105.41 0) (unit 1)
     (in_bom yes) (on_board yes) (fields_autoplaced)
-    (property "Reference" "#PWR0412" (id 0) (at 186.69 111.76 0)
-      (effects (font (size 1.27 1.27)) hide)
-    )
+    (property "Reference" "#PWR0253" (id 0) (at 186.69 111.76 0)
+      (effects (font (size 1.27 1.27)) hide)
+    )

Commit message: BoM
Parts:
- D55, D56, D57, D58, D59: DigiKey Price/Stock (none) -> https://www.digikey.co.uk/en/products/detail/w%C3%BCrth-ele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; Height (none) -> 2
- K50, K51: value ~ -> G6K-2P DC12; DigiKey Price/Stock (none) -> https://www.digikey.co.uk/en/products/detail/omron-electron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; Manufacture Omron Electronics Inc-EMC Div -> (none); Manufacturer (none) -> Omron Electronics Inc-EMC Div

Commit message: changes
Parts:
- removed D58, D59: Green, Diode_SMD:D_1206_3216Metric_Pad1.42x1.75mm_HandSolder, symbol Device:LED_Small_Filled
- removed R85, R86: 1k2, Resistor_SMD:R_1206_3216Metric_Pad1.30x1.75mm_HandSolder, symbol Device:R_Small
- K50, K51: value G6K-2P DC12 -> PC357; footprint Relay_THT:Relay_DPDT_Omron_G6K-2P -> _Connectors:PC375; DigiKey # Z117-ND -> 2634-PC375-2C-12S4-X-ND; DigiKey Price/Stock https://www.digikey.co.uk/en/products/detail/omron-electron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 -> https://www.digikey.co.uk/en/products/detail/picker-compone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; Manufacturer Omron Electronics Inc-EMC Div -> Picker Components; Manufacturer # G6K-2P DC12 -> PC375-2C-12S4-X
Connections:
- net RAG Amber and Red: now reaches K50.2, K51.3
- net RAG Green only: now reaches K50.4, K51.6
