File: CIB_Main_PCB - Mimic Octopus/Volt Free Contacts.kicad_sch (KiCad schematic)
At the start: 28 parts, among them J3 VFC 1-2, J4 VFC 3-4, J5 VFC 5-6, J6 VFC 7-8

Commit message: added changes
Parts:
- J4: renamed from J3; footprint Component Search Engine:Pluggable Terminal Blocks SDDC 1,5 6-PV-3,5 -> Component Search Engine:Pluggable Terminal Blocks SDDC 1.5mm pitch 12 Pin
- J5: renamed from J4; footprint Component Search Engine:Pluggable Terminal Blocks SDDC 1,5 6-PV-3,5 -> Component Search Engine:Pluggable Terminal Blocks SDDC 1.5mm pitch 12 Pin
- J6: renamed from J5; footprint Component Search Engine:Pluggable Terminal Blocks SDDC 1,5 6-PV-3,5 -> Component Search Engine:Pluggable Terminal Blocks SDDC 1.5mm pitch 12 Pin
- J7: renamed from J6; footprint Component Search Engine:Pluggable Terminal Blocks SDDC 1,5 6-PV-3,5 -> Component Search Engine:Pluggable Terminal Blocks SDDC 1.5mm pitch 12 Pin
- renumbered D5 to D10, D6 to D11, D7 to D12, D8 to D13, D1 to D6, D2 to D7, D3 to D8, D4 to D9, K6 to K10, K7 to K11, K8 to K12, K1 to K5, K2 to K6, K3 to K7, K4 to K8, K5 to K9, R5 to R27, R6 to R28, R7 to R29, R8 to R30, R9 to R31, R10 to R32, R11 to R33, R12 to R34

Commit message: BoM
Parts:
- D10, D11, D12, D13, D6, D7, D8, D9: DigiKey Price/Stock (none) -> https://www.digikey.co.uk/en/products/detail/w%C3%BCrth-ele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; Height (none) -> 2
- J4, J5, J6, J7: Mouser # (none) -> 651-1848684; Mouser Part Number 651-1848684 -> (none)
- K10, K11, K12, K5, K6, K7, K8, K9: value ~ -> G6K-2P DC12; DigiKey Price/Stock (none) -> https://www.digikey.co.uk/en/products/detail/omron-electron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; Manufacture Omron Electronics Inc-EMC Div -> (none); Manufacturer (none) -> Omron Electronics Inc-EMC Div

Commit message: changes
Parts:
- removed D10, D11, D12, D13, D6, D7, D8, D9: Green, Diode_SMD:D_1206_3216Metric_Pad1.42x1.75mm_HandSolder, symbol Device:LED_Small_Filled
- removed R27, R28, R29, R30, R31, R32, R33, R34: 1k2, Resistor_SMD:R_1206_3216Metric_Pad1.30x1.75mm_HandSolder, symbol Device:R_Small
- K10, K11, K12, K5, K6, K7, K8, K9: value G6K-2P DC12 -> PC357; footprint Relay_THT:Relay_DPDT_Omron_G6K-2P -> _Connectors:PC375; DigiKey # Z117-ND -> 2634-PC375-2C-12S4-X-ND; DigiKey Price/Stock https://www.digikey.co.uk/en/products/detail/omron-electron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 -> https://www.digikey.co.uk/en/products/detail/picker-compone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; Manufacturer Omron Electronics Inc-EMC Div -> Picker Components; Manufacturer # G6K-2P DC12 -> PC375-2C-12S4-X
